File: circuit/aleph-dev/aleph-primary130315.brd (EAGLE design)
At the start: 370.8 x 111.8 mm, 476 parts, among them IC1 AD8606, IC2 AD8606, IC3 AD8606, IC4 AD8606, IC5 AD8606, IC6 AD8606, IC7 AD8607R, IC8 AD8606, IC9 AD8567, J1 SJ1-3533NG, J10 PHA2U, J11 NSJ12HF, J12 NSJ12HF, J15 STX-3680, J16 STX-3680, J17 STX-3680, J18 STX-3680, J19 STX-3680, J2 PJ-102AH/BH, J20 STX-3680, J21 STX-3680, J22 STX-3680, J3 STEREOSW2GND, J4 NSJ12HF, J5 NSJ12HF, J6 STEREOSW2GND, J7 STEREOSW2GND, J8 USBA-VERT, K0 PVA1, K1 PVA1, K2 PVA1, K3 PVA1, P1 M-2X14-DIL-100, P2 M-2X14-DIL-100, P3 M-2X09-DIL-100, P4 M-2X09-DIL-100, P5 EVJ-POT, P6 EVJ-POT, P7 EVJ-POT, P8 EVJ-POT, U1 AT32UC3A0512, U10 LM4040M3, U14 AD1939, U17 AD5686R, U18 FDS9431A, U19 74HC14D, U2 FT232RL, U20 SN74LVC2G14, U21 LM2674, U22 BAS70-04, U23 BAS70-04, U24 BAS70-04, U25 BAS70-04, U3 CY62167EV30-Z, U4 TPS2020, U5 AD7923, U6 LM2678, U7 ADP3339, U8 ADP3339, U9 MT48LC32M16A2tg-75, Y1 12mhz, Y2 ASFL1-27mhz, Y3 ASFL1-12.288mhz

Commit message: march 2013 build
Parts:
- removed C125, C126, C178, C34, C60, C61, C62, C63, C68, C70, C72: 100n, rc-master-smd:C0603
- removed C127, C128, C69, C71: 10u, rc-master-smd:C1206/T
- removed C55, C56, C57, C58, C59: 1u, rc-master-smd:C0603
- removed C64, C65, C66, C67: 10n, rc-master-smd:C0603
- removed D3, D4, D5, D6: 1N4148W-7, diode:SOD123
- removed IC9: AD8567, analog-devices:TSSOP14
- removed J15, J16, J17, J18, J19, J20, J21, J22: STX-3680, monome-inc:STX-3680
- removed JP4: OLED, pinhead:1X20
- removed K0, K1, K2, K3, KM: PVA1, monome-inc:PVA1
- removed L10: 600, rc-master-smd:L1206
- removed LED1: (no value), led:CHIPLED_1206
- removed LED10, LED11, LED12, LED5, LED6, LED7, LED8, LED9: (no value), led:CHIPLED_0805
- removed P2: M-2X14-DIL-100, con-headers-jp:DIL-100-2X14
- removed P4: M-2X09-DIL-100, con-headers-jp:DIL-100-2X09
- removed P5, P6, P7, P8: EVJ-POT, monome-inc:EVJ-POT
- removed R146, R147, R148, R149, R150, R151, R152, R153, R51, R52, R53, R54, R55, R56, R57, R58, R59, R60, R61, R62: 10k, rc-master-smd:R0603
- removed R2, R29, R30, R32, R34: 82k, rc-master-smd:R0603
- removed R21: 150, rc-master-smd:R0603
- removed R28, R3, R31, R33, R35: 18k, rc-master-smd:R0603
- removed R67: 1k, rc-master-smd:R0603
- removed U$10: NHD-2.7, monome-inc:NHD-2.7
- removed U$2, U$3, U$4, U$5: BOURNS-EM14, monome-inc:BOURNS-EM14
- removed U10: LM4040M3, diode:SOT23
- removed U19: 74HC14D, 74xx-us:SO14
- removed U22, U23, U24, U25: BAS70-04, diode:SOT23
- removed U5: AD7923, monome-inc:TSSOP16
- C18: device rc-master-smd:C1206 -> rc-master-smd:C0603
- C43: device rc-master-smd:C1206/T -> rc-master-smd:C1206
- C46: device rc-master-smd:C3528/T -> rc-master-smd:C3225
- C75: device rc-master-smd:C1210/T -> rc-master-smd:C3528/T
- R36: value 10k -> 100k
- R64: value 47k -> 100k
- moved C18 5.36 mm to (137.8, 62.9), turned to 270 degrees
- moved C13 2.54 mm to (139.1, 69.8)
- moved C9 2.54 mm to (141.0, 69.8)
- moved C17 0.95 mm to (133.7, 66.7)
Connections:
- removed net +5VA: C68.2, C69.+, L10.1, R51.2, R54.2, R57.2, R60.2, R67.1, U22.2, U23.2, U24.2, U25.2, U5.5, U5.6
- removed net CVOUT1^: IC9.3, P4.15
- removed net CVOUT2^: IC9.5, P4.16
- removed net CVOUT3^: IC9.10, P4.18
- removed net CVOUT4^: IC9.12, P4.17
- removed net ENC0A^: P2.7, U$2.P$2
- removed net ENC0B^: P2.8, U$2.P$6
- removed net ENC1A^: P2.5, U$3.P$2
- removed net ENC1B^: P2.6, U$3.P$6
- removed net ENC2A^: P2.3, U$4.P$2
- removed net ENC2B^: P2.4, U$4.P$6
- removed net ENC3A^: P2.1, U$5.P$2
- removed net ENC3B^: P2.2, U$5.P$6
- removed net HP-LP^: P4.10
- removed net HP-L^: P4.9
- removed net HP-RP^: P4.12
- removed net HP-R^: P4.11
- removed net IN1-LP^: P4.6
- removed net IN1-L^: P4.5
- removed net IN1-RP^: P4.8
- removed net IN1-R^: P4.7
- removed net KEY0^: P2.12, U19.8
- removed net KEY1^: P2.11, U19.10
- removed net KEY2^: P2.10, U19.12
- removed net KEY3^: P2.9, U19.2
- removed net MODE-KEY^: P2.13, U19.4
- removed net MODE-LED^: P2.14, R21.1
- removed net N$1: IC9.2, R146.1, R147.2
- removed net N$10: K1.1, K1.4, R28.1, R29.2
- removed net N$11: C56.2, R28.2, U19.11
- removed net N$116: C65.1, R55.1, R56.1, U23.3, U5.11
- removed net N$117: C66.1, R58.1, R59.1, U24.3, U5.10
- removed net N$118: C67.1, R61.1, R62.1, U25.3, U5.9
- removed net N$119: C64.1, R52.1, R53.1, U22.3, U5.12
- removed net N$132: IC9.6, R148.1, R149.2
- removed net N$135: IC9.9, R150.1, R151.2
- removed net N$136: IC9.13, R152.1, R153.2
- removed net N$137: IC9.8, J19.4, R151.1
- removed net N$138: IC9.14, J20.4, R153.1
- removed net N$139: IC9.7, J22.4, R149.1
- removed net N$2: K0.1, K0.4, R2.2, R3.1
- removed net N$20: LED1.C, R21.2
- removed net N$21: K2.1, K2.4, R30.2, R31.2
- removed net N$23: C57.2, R31.1, U19.13
- removed net N$27: K3.1, K3.4, R32.2, R33.2
- removed net N$30: C58.2, R33.1, U19.1
- removed net N$33: J17.1, R57.1
- removed net N$34: D3.A, J15.4
- removed net N$37: D4.C, R55.2
- removed net N$39: D3.C, R52.2
- removed net N$40: D5.C, R58.2
- removed net N$41: J16.1, R54.1
- removed net N$42: D4.A, J16.4
- removed net N$43: KM.1, KM.4, R34.2, R35.2
- removed net N$46: D6.C, R61.2
- removed net N$47: J15.1, R51.1
- removed net N$48: D5.A, J17.4
- removed net N$49: C59.2, R35.1, U19.3
- removed net N$51: J18.1, R60.1
- removed net N$52: D6.A, J18.4
- removed net N$56: IC9.1, J21.4, R147.1
- removed net N$58: C72.2, R67.2, U10.1, U5.7
- removed net N$8: C55.2, R3.2, U19.9
- removed net OLED-DC^: JP4.4, P2.15
- removed net OLED-RES^: JP4.16, P2.16
- removed net OUT1-LP^: P4.2
- removed net OUT1-L^: P4.1
- removed net OUT1-RP^: P4.4
- removed net OUT1-R^: P4.3
- removed net SPI1-CS0^: JP4.17, P2.17
- removed net SPI1-CS1^: P2.18, U5.3
- removed net SPI1-MISO^: P2.20, U5.14
- removed net SPI1-MOSI^: JP4.8, P2.21, U5.2
- removed net SPI1-SCK^: JP4.7, P2.22, U5.1
- net +12V: no longer C178.1, IC9.4, P2.24
- net +3V3: no longer C125.2, C127.+, C70.2, C71.+, JP4.2, LED1.A, P2.25, U5.15
- net +5V: now also C46.1; no longer C126.2, C128.+, C34.2, C46.-, C60.2, C61.2, C62.2, C63.2, L10.2, P2.26, R2.1, R29.1, R30.1, R32.1, R34.1, U$2.P$5, U$3.P$5, U$4.P$5, U$5.P$5, U19.14
- net AGND: no longer C178.2, C64.2, C65.2, C66.2, C67.2, C68.1, C69.-, C72.1, IC9.11, J15.3, J15.5, J16.3, J16.5, J17.3, J17.5, J18.3, J18.5, J19.5, J20.5, J21.5, J22.5, P4.13, P4.14, R146.2, R148.2, R150.2, R152.2, R53.2, R56.2, R59.2, R62.2, U10.2, U22.1, U23.1, U24.1, U25.1, U5.13, U5.16, U5.4, U5.8
- net GND: now also C43.1, C46.2; no longer C125.1, C126.1, C127.-, C128.-, C34.1, C43.-, C46.+, C55.1, C56.1, C57.1, C58.1, C59.1, C60.1, C61.1, C62.1, C63.1, C70.1, C71.-, JP4.1, JP4.10, JP4.11, JP4.12, JP4.13, JP4.14, JP4.19, JP4.20, JP4.5, JP4.6, K0.2, K0.3, K1.2, K1.3, K2.2, K2.3, K3.2, K3.3, KM.2, KM.3, P2.23, P2.27, P2.28, U$2.P$1, U$3.P$1, U$4.P$1, U$5.P$1, U19.5, U19.7
- net UNREG_IN: now also C43.2; no longer C43.+
Routing:
- net +3V3: track 418.2 -> 47.5 mm, vias 15 -> 11
- net +5V: track 671.0 -> 303.3 mm, vias 20 -> 14
- net +5VA: track 232.6 -> 0.00 mm, vias 2 -> 0
- net CVOUT4^: track 217.4 -> 0.00 mm, vias 2 -> 0
- net CVOUT1^: track 213.6 -> 0.00 mm
- net CVOUT3^: track 210.9 -> 0.00 mm
- net CVOUT2^: track 208.0 -> 0.00 mm
- net SPI1-SCK^: track 164.6 -> 0.00 mm, vias 4 -> 0
- net SPI1-MOSI^: track 158.3 -> 0.00 mm, vias 4 -> 0
- net OLED-DC^: track 153.5 -> 0.00 mm, vias 2 -> 0
- net OLED-RES^: track 125.5 -> 0.00 mm, vias 2 -> 0
- net SPI1-CS0^: track 119.4 -> 0.00 mm, vias 2 -> 0
- net SPI1-MISO^: track 113.7 -> 0.00 mm, vias 3 -> 0
- net N$49: track 112.8 -> 0.00 mm
- net SPI1-CS1^: track 101.7 -> 0.00 mm, vias 3 -> 0
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- removed copper zone on layer 16, net AGND
- removed copper zone on layer 16, net GND
Other:
- board size 370.8 x 111.8 mm -> 172.7 x 111.8 mm
- board text removed: "130128"
- board text removed: "C"
- board text removed: "GND"
- board text removed: "HPL"
- board text removed: "HPR"
- board text removed: "IN1L"
- board text removed: "IN1R"
- board text removed: "J"
- board text removed: "OUT1L"
- board text removed: "OUT1R"
- board text removed: "aleph/int"
