File: circuit/aleph-dev/aleph.sch (EAGLE design)
At the start: 462 parts, among them IC1 AD8606, IC2 AD8606, IC3 AD8606, IC4 AD8606, IC5 AD8606, IC6 AD8606, IC7 AD8607R, IC8 AD8606, J1 SJ1-3533NG, J10 PHA2U, J11 NSJ12HF, J12 NSJ12HF, J15 STX-3680, J16 STX-3680, J17 STX-3680, J18 STX-3680, J19 STX-3680, J2 PJ-102AH/BH, J20 STX-3680, J21 STX-3680, J22 STX-3680, J3 STEREOSW2GND, J4 NSJ12HF, J5 NSJ12HF, J6 STEREOSW2GND, J7 STEREOSW2GND, J8 USBA-VERT, K0 PVA1, K1 PVA1, K2 PVA1, K3 PVA1, P1 M-2X14-DIL-100, P2 M-2X14-DIL-100, P3 F-2X10-DIL-100, P4 F-2X10-DIL-100, P5 EVJ-POT, P6 EVJ-POT, P7 EVJ-POT, P8 EVJ-POT, U1 AT32UC3A0512, U10 LM4040M3, U14 AD1939, U17 AD5686R, U18 FDS9431A, U19 74HC14D, U2 FT232RL, U20 SN74LVC2G14, U3 CY62167EV30-Z, U4 TPS2020, U5 AD7923, U6 LM2678, U7 ADP3339, U8 ADP3339, U9 MT48LC32M16A2tg-75, Y1 12mhz, Y2 ASFL1-27mhz, Y3 ASFL1-12.288mhz

Commit message: new proto arrived
Parts:
- removed R68, R69: 0, rc-master-smd:R_0603
- added C175: 15u, rc-master-smd:CP_6032
- added C176: 68u, rc-master-smd:CP_7343
- added C177: 10n, rc-master-smd:C_0603
- added C178: 100n, rc-master-smd:C_0603
- added D8: MBRS130LT3, diode:MBRS130LT3
- added IC9: AD8567, analog-devices:AD8544RU
- added L10: 600, rc-master-smd:L_1206
- added L9: LPS4018-68uh, inductor-coilcraft:LPS4018
- added R146, R147, R148, R149, R150, R151, R152, R153: 10k, rc-master-smd:R_0603
- added U21: LM2674, monome-inc:LM2674
- P3, P4: value F-2X10-DIL-100 -> M-2X09-DIL-100; device con-headers-jp:F-2X10-DIL-100 -> con-headers-jp:M-2X09-DIL-100
- renumbered U$11 to U23, U$12 to U24, U$13 to U25, U$7 to U22
Connections:
- removed net N$89: J21.4
- removed net N$90: J22.4
- removed net N$91: J19.4
- removed net N$93: J20.4
- new net +12V: C176.+, C178.1, IC9P.V+, L9.2, P1.24, P2.24, U21.FB
- new net N$132: IC9B.IN-, R148.1, R149.2
- new net N$133: C177.1, U21.CB
- new net N$134: C177.2, D8.C, L9.1, U21.SWITCH
- new net N$135: IC9C.IN-, R150.1, R151.2
- new net N$136: IC9D.IN-, R152.1, R153.2
- new net N$137: IC9C.OUT, J19.4, R151.1
- new net N$138: IC9D.OUT, J20.4, R153.1
- new net N$139: IC9B.OUT, J22.4, R149.1
- new net POWER_ON: J10.0, R162.1, U21.ON/_OFF, U6.ON/_OFF
- new net UNREG_IN: C175.+, C43.2, C44.2, D1.C, R63.2, U21.INPUT, U6.INPUT
- net +5V: now also C120.1, C121.+, L10.2, U17.GAIN, U17.VDD; no longer R68.2
- net +5VA: now also L10.1; no longer C120.1, C121.+, P3.14, P4.14, R68.1, U17.GAIN, U17.VDD
- net AGND: now also C178.2, IC9P.V-, J19.5, J20.5, J21.5, J22.5, P3.14, P4.14, R146.2, R148.2, R150.2, R152.2; no longer P3.15, P3.16, P4.15, P4.16, R69.1
- net CVOUT1: now also P3.15; no longer P3.17
- net CVOUT1^: now also IC9A.IN+, P4.15; no longer P4.17
- net CVOUT2: now also P3.16; no longer P3.18
- net CVOUT2^: now also IC9B.IN+, P4.16; no longer P4.18
- net CVOUT3: now also P3.18; no longer P3.20
- net CVOUT3^: now also IC9C.IN+, P4.18; no longer P4.20
- net CVOUT4: now also P3.17; no longer P3.19
- net CVOUT4^: now also IC9D.IN+, P4.17; no longer P4.19
- net GND: now also C175.-, C176.-, D8.A, P1.23, P2.23, U21.GND; no longer R69.2
- net N$1: now also IC9A.IN-, R146.1, R147.2; no longer C43.2, C44.2, D1.C, R63.2, U6.INPUT
- net N$56: now also IC9A.OUT, J21.4, R147.1; no longer J10.0, R162.1, U6.ON/_OFF
Other:
- moved on the sheet: C38, J19, J20, J21, J22, J6, J7, R40, R41

Commit message: march 2013 build
Parts:
- removed R166: 100k, rc-master-smd:R_0603
- C18: device rc-master-smd:C_0603 -> rc-master-smd:C_1206
- C43: device rc-master-smd:C_1206 -> rc-master-smd:CP_1206/T
- C46: device rc-master-smd:C_3225 -> rc-master-smd:CP_3528
- C75: device rc-master-smd:CP_3528 -> rc-master-smd:CP_1210/T
- R36: value 100k -> 10k
- R64: value 100k -> 47k
Connections:
- net +3V3: now also U3.!BYTE!
- net +3V3C: now also U14.COUT; no longer R166.1
- net +5V: now also C46.-; no longer C46.1
- net B-MISO: no longer U14.COUT
- net B-MOSI: no longer U14.CIN
- net B-SCK: no longer U14.CCLK
- net B-SPISEL4: no longer R166.2, U14._CLATCH
- net GND: now also C43.-, C46.+, U14.CCLK, U14.CIN, U14._CLATCH; no longer C43.1, C46.2, U3.!BYTE!
- net UNREG_IN: now also C43.+; no longer C43.2

Commit message: arrived
Parts:
- removed C140: 100n, rc-master-smd:C_0603
- removed C141, C160: 330p, rc-master-smd:C_0603
- removed C155, C161: 680p, rc-master-smd:C_0603
- removed C156, C162: 100p, rc-master-smd:C_0603
- removed C157, C163: 220p, rc-master-smd:C_0603
- removed C158, C164: 2200p, rc-master-smd:C_0603
- removed C159, C165: 10u, rc-master-smd:CP_1206/T
- removed IC4: AD8606, analog-devices:AD8607R
- removed R117, R124: 11k, rc-master-smd:R_0603
- removed R118, R120, R125, R127: 5k49, rc-master-smd:R_0603
- removed R119, R126: 3k32, rc-master-smd:R_0603
- removed R121, R128: 604, rc-master-smd:R_0603
- removed R122, R129: 1k65, rc-master-smd:R_0603
- removed R123, R130: 49k9, rc-master-smd:R_0603
- removed R131, R132: 2k74, rc-master-smd:R_0603
Connections:
- removed net N$102: C141.2, R117.1, R119.2, R120.2
- removed net N$103: C155.1, R118.1, R122.1, R131.1
- removed net N$107: C157.2, IC4A.IN+, R122.2
- removed net N$109: C156.2, IC4A.OUT, R120.1, R121.1
- removed net N$111: C158.2, C159.+, R121.2
- removed net N$112: C156.1, IC4A.IN-, R119.1
- removed net N$113: C160.2, R124.1, R126.2, R127.2
- removed net N$114: C161.1, R125.1, R129.1, R132.1
- removed net N$115: C163.2, IC4B.IN+, R129.2
- removed net N$120: C162.2, IC4B.OUT, R127.1, R128.1
- removed net N$121: C164.2, C165.+, R128.2
- removed net N$122: C162.1, IC4B.IN-, R126.1
- net +3V3A: no longer C140.2, IC4P.V+
- net +5V: now also C46.+; no longer C46.-
- net AGND: no longer C140.1, C141.1, C155.2, C157.1, C158.1, C160.1, C161.2, C163.1, C164.1, IC4P.V-, R123.2, R130.2
- net GND: now also C46.-; no longer C46.+
- net HP-LP: no longer C165.-, R130.1
- net HP-RP: no longer C159.-, R123.1
- net HPL+: no longer R125.2
- net HPL-: no longer R124.2
- net HPR+: no longer R118.2
- net HPR-: no longer R117.2
- net VREF: no longer R131.2, R132.2
Other:
- moved on the sheet: C46

Commit message: todos
Parts:
- R162: value 100k -> 1k
Changed lines of the file:
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@@
 <part name="V57" library="supply" deviceset="+5VA" device=""/>
 <part name="GND66" library="supply" deviceset="GND" device=""/>
-<part name="R162" library="rc-master-smd" deviceset="R_" device="0603" value="100k"/>
+<part name="R162" library="rc-master-smd" deviceset="R_" device="0603" value="1k"/>
 <part name="GND5" library="supply" deviceset="GND" device=""/>
 <part name="U3" library="memory-cypress" deviceset="CY62167EV30-Z" device=""/>

Commit message: up
Parts:
- added U$7, U$8: TOGGLE, monome-inc:TOGGLE
Other:
- note removed: "note: r67 and r68 matched. 1%"
Changed lines of the file:
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@@
 <part name="L10" library="rc-master-smd" deviceset="L_" device="1206" value="600"/>
 <part name="GND4" library="supply" deviceset="GND" device=""/>
+<part name="U$7" library="monome-inc" deviceset="TOGGLE" device=""/>
+<part name="U$8" library="monome-inc" deviceset="TOGGLE" device=""/>
 </parts>
 <sheets>
@@
 <wire x1="299.72" y1="35.56" x2="299.72" y2="266.7" width="0.1524" layer="97"/>
 <wire x1="142.24" y1="152.4" x2="401.32" y2="152.4" width="0.1524" layer="97"/>
-<text x="38.1" y="246.38" size="1.778" layer="97">note: r67 and r68 matched. 1%</text>
 <text x="396.24" y="83.82" size="5.08" layer="97" rot="R180">I2C</text>
 <text x="398.78" y="264.16" size="5.08" layer="97" rot="R180">OLED</text>
@@
 <instance part="R174" gate="G$1" x="248.92" y="109.22" rot="R180"/>
 <instance part="AGND63" gate="VR1" x="242.57" y="102.87"/>
+<instance part="U$7" gate="G$1" x="149.86" y="53.34"/>
+<instance part="U$8" gate="G$1" x="147.32" y="25.4"/>
 </instances>
 <busses>

Commit message: new face
Parts:
- removed U$8: TOGGLE, monome-inc:TOGGLE
- added C140, C141, C156, C157, C159, C160, C196, C197, C207, C208, C210, C211: 10u, rc-master-smd:CP_1206/T
- added C155, C158, C161, C192, C193, C194, C195, C198, C209: 100n, rc-master-smd:C_0603
- added C162, C164, C165: 100u, rc-master-smd:CP_1206/T
- added C163, C191: 1u, rc-master-smd:C_0603
- added IC10, IC11, IC12, IC13, IC14, IC4: AD8607R, analog-devices:AD8607R
- added J13: PHA2U, monome-inc:PHA2U
- added R117, R119, R120, R121, R122, R123, R124, R126, R127, R128, R156, R157, R158, R159, R160, R161, R166, R176, R177, R178, R179, R180, R181, R183, R184, R185, R68, R69: 100k, rc-master-smd:R_0603
- added R118, R125, R175, R182: 50k, rc-master-smd:R_0603
- added R129, R130, R132, R154: 3k9, rc-master-smd:R_0603
- added R131, R155: 5k, rc-master-smd:R_0603
- added R186, R187: 5M, rc-master-smd:R_0603
- U$7: value TOGGLE -> (none); device monome-inc:TOGGLE -> monome-inc:TDA1308
Connections:
- removed net HP-LP: P3.10
- removed net HP-LP^: P4.10
- removed net HP-RP: P3.12
- removed net HP-RP^: P4.12
- new net GAINL-1: IC14B.IN-, J13._0, R182.2
- new net GAINL-2: C208.+, IC14B.OUT, R181.2, R187.2
- new net GAINR-1: IC13B.IN-, J13.0, R175.2
- new net GAINR-2: C197.+, IC13B.OUT, R166.2, R186.2
- new net IN-VREF: IC12A.IN-, IC12A.OUT, P7.2, P7.3, P8.2, P8.3, R176.1, R177.1, R183.1, R184.1
- new net N$102: C156.-, R118.1
- new net N$103: IC4B.IN-, R117.1, R118.2
- new net N$107: C141.+, IC4B.OUT, R117.2
- new net N$109: IC10A.IN+, R127.2
- new net N$111: IC4B.IN+, R119.2
- new net N$112: P5.1, R68.1
- new net N$113: IC10A.IN-, R122.2, R123.1
- new net N$114: C159.+, IC10A.OUT, R123.2
- new net N$115: C159.-, R125.1
- new net N$120: IC10B.IN-, R124.1, R125.2
- new net N$121: C157.+, IC10B.OUT, R124.2
- new net N$122: IC10B.IN+, R126.2
- new net N$130: P5.4, R122.1
- new net N$140: C160.+, P5.5
- new net N$141: R129.1, R130.2, U$7.INA-
- new net N$148: C164.+, R129.2, U$7.OUTA
- new net N$149: C163.1, P6.5
- new net N$150: R132.2, R154.1, U$7.INB-
- new net N$151: C191.1, P6.6
- new net N$152: C192.2, IC12A.IN+, R156.1, R157.2
- new net N$153: IC13A.IN+, R177.2
- new net N$154: C165.-, R132.1, U$7.OUTB
- new net N$155: IC13A.IN-, R160.2, R161.1
- new net N$156: P6.4, R154.2
- new net N$157: P6.1, R130.1
- new net N$158: C207.+, IC13A.OUT, R161.2
- new net N$159: C207.-, R175.1
- new net N$162: IC13B.IN+, R176.2
- new net N$163: C193.2, IC12B.IN+, R158.1, R159.2
- new net N$164: C196.+, P8.6
- new net N$165: P8.1, R160.1
- new net N$166: IC14A.IN+, R184.2
- new net N$167: IC14A.IN-, R179.2, R180.1
- new net N$168: C210.+, IC14A.OUT, R180.2
- new net N$169: C210.-, R182.1
- new net N$172: IC14B.IN+, R183.2
- new net N$173: P7.1, R179.1
- new net N$174: C211.+, P7.6
- new net N$177: J13.1, R166.1
- new net N$180: J13.2, R186.1
- new net N$181: J13._1, R181.1
- new net N$183: J13._2, R187.1
- new net N$89: IC4A.IN+, R120.2
- new net N$90: IC4A.IN-, R68.2, R69.1
- new net N$91: C140.+, P5.6
- new net N$93: C156.+, IC4A.OUT, R69.2
- new net OUT-VREF: IC12B.IN-, IC12B.OUT, P5.2, P5.3, P6.2, P6.3, R119.1, R120.1, R126.1, R127.1, U$7.INA+, U$7.INB+
- new net OUT1-LB: C160.-, C163.2, IC11B.IN-, IC11B.OUT
- new net OUT1-RB: C140.-, C191.2, IC11A.IN-, IC11A.OUT
- net +5VA: now also C155.2, C158.2, C161.2, C162.+, C194.2, C195.2, C198.2, C209.2, IC10P.V+, IC11P.V+, IC12P.V+, IC13P.V+, IC14P.V+, IC4P.V+, R156.2, R158.2, U$7.VDD
- net AGND: now also C155.1, C158.1, C161.1, C162.-, C192.1, C193.1, C194.1, C195.1, C198.1, C209.1, IC10P.V-, IC11P.V-, IC12P.V-, IC13P.V-, IC14P.V-, IC4P.V-, R121.1, R128.1, R131.1, R155.2, R157.1, R159.1, R178.1, R185.1, U$7.VSS
- net HP-L^: now also C165.+, R155.1
- net HP-R^: now also C164.-, R131.2
- net IN1-LP^: now also C211.-
- net IN1-L^: now also C208.-, R185.2
- net IN1-RP^: now also C196.-
- net IN1-R^: now also C197.-, R178.2
- net OUT1-LP^: now also IC11B.IN+
- net OUT1-L^: now also C157.-, R128.2
- net OUT1-RP^: now also IC11A.IN+
- net OUT1-R^: now also C141.-, R121.2
