File: circuit/aleph-dev/aleph.sch (EAGLE design)
At the start: 524 parts, among them IC1 AD8606, IC10 AD8607R, IC12 AD8607R, IC13 AD8607R, IC14 AD8607R, IC15 AD8607R, IC2 AD8606, IC3 AD8606, IC5 AD8606, IC6 AD8606, IC7 AD8607R, IC8 AD8606, IC9 AD8567, J1 SJ1-3533NG, J10 PHA2U, J11 NSJ12HF, J12 NSJ12HF, J13 PHA2U, J14 F-2X03-DIL-100, J15 STX-3680, J16 STX-3680, J17 STX-3680, J18 STX-3680, J19 STX-3680, J2 PJ-102AH/BH, J20 STX-3680, J21 STX-3680, J22 STX-3680, J3 STEREOSW2GND, J4 NSJ12HF, J5 NSJ12HF, J6 STEREOSW2GND, J7 STEREOSW2GND, J8 USBA-VERT, K0 PVA1, K1 PVA1, K2 PVA1, K3 PVA1, P1 M-2X14-DIL-100, P10 M-1X05-SIP-100-32, P2 M-2X14-DIL-100, P3 F-2X06-DIL-100, P4 M-2X06-DIL-100, P5 EVJ-POT, P6 EVJ-POT, P7 EVJ-POT, P8 EVJ-POT, P9 M-2X03-DIL-100, U1 AT32UC3A0512, U10 LM4040M3, U12 BAS70-04, U13 BAS70-04, U14 AD1939, U17 AD5686R, U18 FDS9431A, U19 74HC14D, U20 SN74LVC2G14, U22 BAS70-04, U23 BAS70-04, U24 BAS70-04, U25 BAS70-04, U3 CY62167EV30-Z, U4 TPS2020, U5 AD7923, U6 LM2678, U7 ADP3339, U8 ADP3339, U9 MT48LC32M16A2tg-75, X1 16mhz, Y1 12mhz, Y2 ASFL1-27mhz, Y3 ASFL1-12.288mhz

Commit message: almost final circuit
Parts:
- removed IC14, IC15: AD8607R, analog-devices:AD8607R
- removed JP4: OLED, pinhead:PINHD-1X20
- removed K0: PVA1, monome-inc:PVA1
- removed L11: XAL7030-103, monome-inc:XAL7030-103
- removed U$7: TPA6111A2, monome-inc:TPA6111A2
- removed U$8: ATMEGA32U4-AU, monome-inc:ATMEGA32U4-AU
- added C215, C223, C226: 100n, rc-master-smd:C_0603
- added C219: 2200p, rc-master-smd:C_0603
- added C220, C221: 1n, rc-master-smd:C_0603
- added C222: 470n, rc-master-smd:C_1206
- added C224: 330p, rc-master-smd:C_0603
- added C225, C227: 10u, rc-master-smd:CP_1206/T
- added C228: 220p, rc-master-smd:C_0603
- added C52: 100u, rc-master-smd:CP_1210/T
- added D10, D11, D12, D8: 1N4148W-7, diode:1N4148W-7
- added D13, D14: MBRS360T3, diode:MBRS360T3
- added IC11: AD8607R, analog-devices:AD8607R
- added IC4: AD8606, analog-devices:AD8607R
- added JP2: AVR-JTAG, atmel-avr32:AVR-JTAG-10
- added K4: PVA1, monome-inc:PVA1
- added L9: 600, rc-master-smd:L_1206
- added LED5, LED6: (no value), led:LEDCHIPLED_0805
- added LED8: (no value), led:LEDCHIPLED_1206
- added R117, R131: 5k76, rc-master-smd:R_0603
- added R118: 33, rc-master-smd:R_0603
- added R119, R120: 470k, rc-master-smd:R_0603
- added R123, R125, R127, R128: 100k, rc-master-smd:R_0603
- added R124: 56k, rc-master-smd:R_0603
- added R126: 562, rc-master-smd:R_0603
- added R155: 82k, rc-master-smd:R_0603
- added R166, R193, R195, R196: 10k, rc-master-smd:R_0603
- added R167, R168: 39, rc-master-smd:R_0603
- added R181, R186: 49k9, rc-master-smd:R_0603
- added R187: 47k, rc-master-smd:R_0603
- added R188: 330k, rc-master-smd:R_0603
- added R189, R190: 22, rc-master-smd:R_0603
- added R191: 1k, rc-master-smd:R_0603
- added R192: 117k, rc-master-smd:R_0603
- added R194: 13k3, rc-master-smd:R_0603
- added U11: BAS70-04, diode:BAS70-04
- added U15: AT32UC3A0512, atmel-avr32:AT32UC3A0128/0256/0512
- added U16: CY62167EV30-Z, memory-cypress:CY62167EV30-Z
- added U21: AD7923, monome-inc:AD7923
- added U26: SN74LVC2G14, monome-inc:SN74LVC2G14
- C1, C161: value 100n -> 2.2u; device rc-master-smd:C_0603 -> rc-master-smd:C_1206
- C10: value 33n -> 4.7u; device rc-master-smd:C_0603 -> rc-master-smd:CP_1206/T
- C100: value 47u -> 10u
- C101, C120, C143, C145, C34, C63, C70, C8, C81, C82, C83, C84: value 100n -> 10u; device rc-master-smd:C_0603 -> rc-master-smd:CP_1206/T
- C102: value 10u -> 390p; device rc-master-smd:CP_1206/T -> rc-master-smd:C_0603
- C103: value 100n -> 5600p
- C104, C110, C122, C95: value 330p -> 100n
- C105: value 680p -> 10u; device rc-master-smd:C_0603 -> rc-master-smd:CP_1206/T
- C106: value 100p -> 120p
- C107: value 220p -> 100n
- C108, C114, C130: value 2200p -> 100n
- C109, C115, C121, C155, C157, C158, C162, C186, C208, C71, C76, C78: value 10u -> 100n; device rc-master-smd:CP_1206/T -> rc-master-smd:C_0603
- C11, C12, C21: value 33n -> 100p
- C111, C123, C98: value 680p -> 100n
- C112, C116, C124: value 100p -> 1u
- C113, C117: value 220p -> 1u
- C118: value 2200p -> 1u
- C119: value 10u -> 1u; device rc-master-smd:CP_1206/T -> rc-master-smd:C_0603
- C125, C126, C142, C193, C195, C50: value 100n -> 10n
- C127, C128, C140, C156, C48, C49: value 10u -> 10n; device rc-master-smd:CP_1206/T -> rc-master-smd:C_0603
- C129: value 220p -> 10n
- C13: value 33n -> 1u
- C132: value 4.7u -> 10n; device rc-master-smd:CP_1206/T -> rc-master-smd:C_0603
- C133: value 100p -> 10n
- C134, C141: value 100n -> 1n
- C135: value 120p -> 100p
- C136, C150: value 120p -> 100n
- C137, C171, C172, C204: value 1n -> 100n
- C138, C152: value 1n -> 10n
- C139, C148, C154, C173: value 100p -> 100n
- C14: value 4.7u -> 10u; device rc-master-smd:C_1206 -> rc-master-smd:CP_1206/T
- C146: value 100n -> 18p
- C147: value 4.7u -> 18p; device rc-master-smd:CP_1206/T -> rc-master-smd:C_0603
- C149: value 100n -> 4.7u; device rc-master-smd:C_0603 -> rc-master-smd:CP_1206/T
- C15: value 33n -> 100n
- C151: value 120p -> 10n
- C153: value 1n -> 4.7u; device rc-master-smd:C_0603 -> rc-master-smd:C_1206
- C16: value 100n -> 680p
- C163, C191: value 1u -> 33n
- C164: value 68u -> 100n; device rc-master-smd:CP_1206/T -> rc-master-smd:C_0603
- C165: value 68u -> 33n; device rc-master-smd:CP_1206/T -> rc-master-smd:C_0603
- C166, C199: value 4.7u -> 2.7n; device rc-master-smd:CP_1206/T -> rc-master-smd:C_0603
- C167, C200: value 100p -> 33n
- C168, C189: value 100n -> 33n
- C169, C202: value 120p -> 10u; device rc-master-smd:C_0603 -> rc-master-smd:CP_1206/T
- C17: value 4.7u -> 100n; device rc-master-smd:C_1206 -> rc-master-smd:C_0603
- C170: value 120p -> 1n
- C174, C217, C41, C60, C61, C72: value 100n -> 100p
- C175: value 10u -> 330p; device rc-master-smd:CP_1206/T -> rc-master-smd:C_0603
- C176: value 2.2u -> 2200p; device rc-master-smd:C_1206 -> rc-master-smd:C_0603
- C177: value 220p -> 2200p
- C178, C209: value 100n -> 330p
- C179: value 10n -> 33n
- C18: value 2.2u -> 120p; device rc-master-smd:C_1206 -> rc-master-smd:C_0603
- C180: value 10n -> 1n
- C181: value 10n -> 2.2u; device rc-master-smd:C_0603 -> rc-master-smd:C_1206
- C182: value 10n -> 2.7n
- C183, C67: value 10n -> 100n
- C185: value 100u -> 10n; device rc-master-smd:CP_1210/T -> rc-master-smd:C_0603
- C187: value 5600p -> 100n
- C188: value 390p -> 100n
- C19: value 470p -> 100n
- C190, C210, C211, C3: value 10u -> 4.7u
- C192: value 100n -> 2.7n
- C194: value 12p -> 2.7n
- C196: value 10u -> 470p; device rc-master-smd:CP_1206/T -> rc-master-smd:C_0603
- C197, C207: value 10u -> 33n; device rc-master-smd:CP_1206/T -> rc-master-smd:C_0603
- C2: device rc-master-smd:C_1206 -> rc-master-smd:C_0603
- C20: value 2.7n -> 120p
- C201, C6: device rc-master-smd:C_0603 -> rc-master-smd:C_1206
- C203: value 120p -> 4.7u; device rc-master-smd:C_0603 -> rc-master-smd:C_1206
- C205: value 1n -> 33n
- C206: value 100p -> 2.2u; device rc-master-smd:C_0603 -> rc-master-smd:C_1206
- C212: value 1u -> 2200p
- C213: value 1u -> 1n
- C214: value 12p -> 1n
- C216, C38, C59: value 1u -> 100p
- C218: value 4.7u -> 22u
- C22: value 2.2u -> 220p; device rc-master-smd:C_1206 -> rc-master-smd:C_0603
- C23: value 2.7n -> 100n; device rc-master-smd:C_0603 -> rc-master-smd:C_1206
- C24, C25: value 2.7n -> 10u; device rc-master-smd:C_0603 -> rc-master-smd:CP_1206/T
- C26: value 2.7n -> 100n
- C27: value 33n -> 10n; device rc-master-smd:C_0603 -> rc-master-smd:C_1206
- C28: value 33n -> 47u; device rc-master-smd:C_0603 -> rc-master-smd:CP_3528
- C29, C30: value 33n -> 12p
- C31: value 100n -> 1u
- C32: value 18p -> 100n
- C33: value 18p -> 1u
- C35, C64, C65, C66: value 10n -> 10u; device rc-master-smd:C_0603 -> rc-master-smd:CP_1206/T
- C36: value 1u -> 680p
- C37, C97: value 10n -> 120p
- C39, C62: value 100n -> 120p
- C40: value 2.2u -> 100p; device rc-master-smd:C_1206 -> rc-master-smd:C_0603
- C42, C85, C86: value 10n -> 220p
- C43: value 22u -> 1u; device rc-master-smd:CP_1206/T -> rc-master-smd:C_0603
- C44: value 470n -> 1u; device rc-master-smd:C_1206 -> rc-master-smd:C_0603
- C45: value 10n -> 10u; device rc-master-smd:C_1206 -> rc-master-smd:CP_1206/T
- C46: value 47u -> 10u; device rc-master-smd:CP_3528 -> rc-master-smd:CP_1206/T
- C47: value 100n -> 10n; device rc-master-smd:C_1206 -> rc-master-smd:C_0603
- C5: value 33n -> 10u; device rc-master-smd:C_0603 -> rc-master-smd:CP_1206/T
- C51: value 4.7u -> 100u; device rc-master-smd:CP_1206/T -> rc-master-smd:CP_1210/T
- C55: value 1u -> 100n
- C56, C57, C58: value 1u -> 10u; device rc-master-smd:C_0603 -> rc-master-smd:CP_1206/T
- C7, C9: value 100n -> 68u; device rc-master-smd:C_0603 -> rc-master-smd:CP_1206/T
- C73: value 10u -> 100p; device rc-master-smd:CP_1206/T -> rc-master-smd:C_0603
- C74: value 100n -> 10u; device rc-master-smd:C_1206 -> rc-master-smd:CP_1206/T
- C75: value 100u -> 10u; device rc-master-smd:CP_1210/T -> rc-master-smd:CP_1206/T
- C77: value 10u -> 120p; device rc-master-smd:CP_1206/T -> rc-master-smd:C_0603
- C79: value 100n -> 47u; device rc-master-smd:C_0603 -> rc-master-smd:CP_1206/T
- C87, C88, C96: value 10n -> 100p
- C93, C94: value 10n -> 680p
- D1: value MBRS360T3 -> MBR0520L; device diode:MBRS360T3 -> diode:MBR0540
- D2: value MBRS360T3 -> zhcs1000; device diode:MBRS360T3 -> diode:ZENER-DIODESOT23
- D7: value zhcs1000 -> 1N4148W-7; device diode:ZENER-DIODESOT23 -> diode:1N4148W-7
- D9: value MBR0520L -> 1N4148W-7; device diode:MBR0540 -> diode:1N4148W-7
- IC1: value AD8606 -> AD8567; device analog-devices:AD8607R -> analog-devices:AD8544RU
- IC10, IC12: value AD8607R -> AD8606
- IC5, IC6, IC8: value AD8606 -> AD8607R
- IC9: value AD8567 -> AD8606; device analog-devices:AD8544RU -> analog-devices:AD8607R
- J1: value SJ1-3533NG -> STEREOSW2GND; device monome-inc:SJ1-3533NG -> Audio Jacks 0.25 inch:STEREOSW2GND
- J11: value NSJ12HF -> USBA-VERT; device monome-inc:NSJ12HF -> monome-inc:USBA-VERT
- J12: value NSJ12HF -> STX-3680; device monome-inc:NSJ12HF -> monome-inc:STX-3680
- J13: value PHA2U -> STX-3680; device monome-inc:PHA2U -> monome-inc:STX-3680
- J14: value F-2X03-DIL-100 -> STX-3680; device con-headers-jp:F-2X03-DIL-100 -> monome-inc:STX-3680
- J2: value PJ-102AH/BH -> NSJ12HF; device con-cuistack:PJ-102AH/BH -> monome-inc:NSJ12HF
- J20: value STX-3680 -> F-2X03-DIL-100; device monome-inc:STX-3680 -> con-headers-jp:F-2X03-DIL-100
- J21, J22: value STX-3680 -> STEREOSW2GND; device monome-inc:STX-3680 -> Audio Jacks 0.25 inch:STEREOSW2GND
- J3: value STEREOSW2GND -> NSJ12HF; device Audio Jacks 0.25 inch:STEREOSW2GND -> monome-inc:NSJ12HF
- J6: value STEREOSW2GND -> SJ1-3533NG; device Audio Jacks 0.25 inch:STEREOSW2GND -> monome-inc:SJ1-3533NG
- J7: value STEREOSW2GND -> (none); device Audio Jacks 0.25 inch:STEREOSW2GND -> monome-inc:USB_TYPE_B
- J8: value USBA-VERT -> PJ-102AH/BH; device monome-inc:USBA-VERT -> con-cuistack:PJ-102AH/BH
- J9: value (none) -> PHA2U; device monome-inc:USB_TYPE_B -> monome-inc:PHA2U
- JP1: value AVR-JTAG -> OLED; device atmel-avr32:AVR-JTAG-10 -> pinhead:PINHD-1X20
- L1: value MSS1278 -> XAL7030-103; device inductor-coilcraft:MSS1278 -> monome-inc:XAL7030-103
- L2: value SRR6038-100Y -> 600; device inductor-bourns:SRR6038 -> rc-master-smd:L_1206
- L4: value 600 -> MSS1278; device rc-master-smd:L_1206 -> inductor-coilcraft:MSS1278
- L8: value 600 -> SRR6038-100Y; device rc-master-smd:L_1206 -> inductor-bourns:SRR6038
- LED1, LED2: device led:LEDCHIPLED_1206 -> led:LEDCHIPLED_0805
- LED12: device led:LEDCHIPLED_0805 -> led:LEDCHIPLED_1206
- P1: value M-2X14-DIL-100 -> M-1X05-SIP-100-32; device con-headers-jp:M-2X14-DIL-100 -> con-headers-jp:M-1X05-SIP-100-32
- P10: value M-1X05-SIP-100-32 -> M-2X03-DIL-100; device con-headers-jp:M-1X05-SIP-100-32 -> con-headers-jp:M-2X03-DIL-100
- P2: value M-2X14-DIL-100 -> EVJ-POT; device con-headers-jp:M-2X14-DIL-100 -> monome-inc:EVJ-POT
- P3: value F-2X06-DIL-100 -> EVJ-POT; device con-headers-jp:F-2X06-DIL-100 -> monome-inc:EVJ-POT
- P4: value M-2X06-DIL-100 -> EVJ-POT; device con-headers-jp:M-2X06-DIL-100 -> monome-inc:EVJ-POT
- P6: value EVJ-POT -> F-2X06-DIL-100; device monome-inc:EVJ-POT -> con-headers-jp:F-2X06-DIL-100
- P7: value EVJ-POT -> M-2X06-DIL-100; device monome-inc:EVJ-POT -> con-headers-jp:M-2X06-DIL-100
- P8: value EVJ-POT -> M-2X14-DIL-100; device monome-inc:EVJ-POT -> con-headers-jp:M-2X14-DIL-100
- P9: value M-2X03-DIL-100 -> M-2X14-DIL-100; device con-headers-jp:M-2X03-DIL-100 -> con-headers-jp:M-2X14-DIL-100
- R10, R11, R14, R159, R161, R176, R179, R69, R8: value 100k -> 10k
- R100: value 49k9 -> 750k
- R101: value 11k -> 10k
- R102: value 5k49 -> 5k76
- R103: value 3k32 -> 5k76
- R104, R94: value 5k49 -> 10k
- R105: value 604 -> 270
- R106: value 1k65 -> 270
- R107: value 49k9 -> 270
- R108, R109: value 2k74 -> 10k
- R110, R169: value 5k76 -> 10k
- R111: value 5k76 -> 2k74
- R112: value 237 -> 2k74
- R113, R114, R143: value 5k76 -> 4k7
- R115: value 237 -> 1k
- R116: value 750k -> 5k76
- R12, R13, R9: value 100k -> 47k
- R121: value 117k -> 470k
- R122: value 13k3 -> 56k
- R129: value 20k -> 750k
- R130: value 20k -> 5k76
- R132: value 20k -> 100k
- R133, R134, R137, R138: value 5k76 -> 100k
- R135: value 237 -> 82k
- R136, R142: value 5k76 -> 18k
- R139, R141, R173: value 237 -> 100k
- R140: value 5k76 -> 0
- R144: value 237 -> 0
- R145: value 750k -> 4k7
- R146, R73: value 10k -> 100k
- R147, R149, R151, R153: value 10k -> 82k
- R148, R150, R152: value 10k -> 18k
- R15: value 22 -> 120
- R154: value 20k -> 18k
- R156: value 100k -> 82k
- R157: value 100k -> 18k
- R158: value 100k -> 150
- R16, R17, R18: value 0 -> 120
- R160: value 100k -> 22
- R162, R67: value 1k -> 10k
- R163, R171, R172: value 5k76 -> 237
- R164: value 562 -> 237
- R170: value 237 -> 10k
- R174: value 750k -> 49k9
- R175: value 50k -> 49k9
- R177, R180: value 100k -> 0
- R178: value 100k -> 33
- R182: value 50k -> 237
- R183, R184, R185: value 100k -> 237
- R19, R20: value 47k -> 120
- R2: value 82k -> 10k
- R21: value 150 -> 11k
- R22: value 22 -> 5k49
- R23, R47: value 150 -> 5k76
- R24, R25, R26, R49, R50: value 0 -> 5k76
- R27: value 3.32k -> 750k
- R28: value 18k -> 750k
- R29: value 82k -> 3k32
- R3: value 18k -> 10k
- R30: value 82k -> 1k65
- R31: value 18k -> 5k49
- R32, R34: value 82k -> 20k
- R33, R35: value 18k -> 20k
- R36, R54: value 10k -> 2k74
- R37: value 22 -> 150
- R38: value 18k -> 150
- R39: value 82k -> 604
- R4, R5: value 39 -> 10k
- R40: value 18k -> 0
- R41: value 82k -> 0
- R43: value 750k -> 0
- R44, R82: value 11k -> 604
- R45: value 5k49 -> 3.32k
- R46: value 3k32 -> 0
- R48, R75: value 10k -> 5k76
- R51: value 47k -> 5k49
- R52: value 10k -> 3k32
- R53: value 10k -> 1k65
- R55, R72: value 10k -> 0
- R56, R58, R59: value 10k -> 270
- R57: value 100k -> 270
- R6: value 0 -> 10k
- R60: value 47k -> 270
- R61: value 10k -> 150
- R63: value 330k -> 10k
- R64: value 47k -> 10k
- R7: value 0 -> 47k
- R70: value 4k7 -> 11k
- R71: value 4k7 -> 5k49
- R74: value 33 -> 100k
- R76: value 33 -> 5k76
- R77: value 150 -> 470k
- R78: value 10k -> 470k
- R79, R80: value 10k -> 4k7
- R81, R84: value 2k74 -> 5k49
- R83: value 5k49 -> 604
- R85: value 3k32 -> 100k
- R86: value 5k49 -> 100k
- R87: value 604 -> 1k
- R88: value 1k65 -> 1k
- R89: value 49k9 -> 11k
- R90: value 11k -> 3k32
- R91: value 5k49 -> 3k32
- R92: value 5k49 -> 11k
- R93: value 3k32 -> 10k
- R95: value 604 -> 10k
- R96, R99: value 1k65 -> 5k49
- R97: value 49k9 -> 1k65
- R98: value 604 -> 1k65
- U1: value AT32UC3A0512 -> BAS70-04; device atmel-avr32:AT32UC3A0128/0256/0512 -> diode:BAS70-04
- U10: value LM4040M3 -> FDS9431A; device diode:LM4040M3 -> monome-inc:FDS9431A
- U14: value AD1939 -> BAS70-04; device monome-inc:AD1939 -> diode:BAS70-04
- U17: value AD5686R -> AD1939; device monome-inc:AD5686R -> monome-inc:AD1939
- U18: value FDS9431A -> TL072D; device monome-inc:FDS9431A -> linear:TL072D
- U19: value 74HC14D -> TL072D; device 74xx-us:74HC14D -> linear:TL072D
- U20: value SN74LVC2G14 -> TL072D; device monome-inc:SN74LVC2G14 -> linear:TL072D
- U22: value BAS70-04 -> LM4040M3; device diode:BAS70-04 -> diode:LM4040M3
- U23: value BAS70-04 -> MT48LC32M16A2tg-75; device diode:BAS70-04 -> monome-inc:MT48LC16M16A2
- U24: value BAS70-04 -> AD5686R; device diode:BAS70-04 -> monome-inc:AD5686R
- U25: value BAS70-04 -> 74HC14D; device diode:BAS70-04 -> 74xx-us:74HC14D
- U3: value CY62167EV30-Z -> BAS70-04; device memory-cypress:CY62167EV30-Z -> diode:BAS70-04
- U5: value AD7923 -> LM2678; device monome-inc:AD7923 -> monome-inc:LM2678
- U6: value LM2678 -> ATMEGA32U4-AU; device monome-inc:LM2678 -> monome-inc:ATMEGA32U4-AU
- U8: value ADP3339 -> TPA6111A2; device monome-inc:ADP3339 -> monome-inc:TPA6111A2
- U9: value MT48LC32M16A2tg-75 -> ADP3339; device monome-inc:MT48LC16M16A2 -> monome-inc:ADP3339
- Y1: value 12mhz -> ASFL1-27mhz; device crystal:CRYTALHC49UP -> crystal:ASFL1
- Y2: value ASFL1-27mhz -> 12mhz; device crystal:ASFL1 -> crystal:CRYTALHC49UP
- renumbered BM0 to BM2, GND0 to TP-GND, JP8 to JP3, U$1 to SW1, U$10 to REF-OLED, U$2 to E1, U$3 to E2, U$4 to E4, U$5 to E3, U$6 to S1, U$9 to U2
Connections:
- removed net N$155: IC13A.IN-, R160.2, R161.1
- new net N$122: J3.TB, R19.1
- new net N$130: J3.RB, R18.1
- new net N$140: J2.TB, R15.1
- new net N$156: J2.RB, R17.1
- new net N$157: J3.TT, R20.1
- new net N$170: J2.TT, R16.1
- new net N$171: J10._2, R12.2
- new net N$175: J10._1, R14.2
- new net N$176: J10.2, R9.2
- new net N$177: J10.1, R5.2
- new net N$178: R58.1, U19B.OUT
- new net N$179: R122.2, R123.1, U19B.+IN
- new net N$180: C64.-, IC7B.IN+
- new net N$181: C58.+, IC7A.IN-
- new net N$182: C64.+, P5.1
- new net N$184: D12.C, D9.A, R121.1, U20A.OUT
- new net N$185: D9.C, R107.2
- new net N$186: C84.+, R107.1, R59.1, R95.1, U20B.-IN
- new net N$187: LED11.A, R110.1, U20A.-IN
- new net N$188: LED6.A, R59.2
- new net N$189: LED7.A, R60.2
- new net N$190: R60.1, U20B.OUT
- new net N$191: R124.2, R125.1, U20B.+IN
- new net N$195: D10.A, R119.2, R87.1, R88.1, U18A.+IN
- new net N$196: D10.C, D7.A, R119.1, U18A.OUT
- new net N$197: D7.C, R105.2
- new net N$198: C82.+, R105.1, R56.1, R93.1
- new net N$199: LED9.A, R108.1, U18A.-IN
- new net N$200: LED3.A, R56.2
- net +12V: now also C10.+, C2.1, C228.2, D1.C, IC1P.V+, P8.24, P9.2, R192.2; no longer C177.2, C178.1, C218.+, D9.C, IC9P.V+, P1.24, P2.2, R121.2
- net +3V3: now also C111.1, C156.1, C195.1, C68.2, C70.+, C81.+, C89.2, JP1.2, JP2.4, LED12.A, LED8.A, P8.25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; no longer C125.2, C127.+, C35.1, C37.1, C41.1, C70.2, C71.+, JP1.4, JP4.2, LED1.A, LED2.A, P1.25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
- net +3V3A: now also C102.1, C107.2, C14.+, C150.1, C160.1, C162.1, C17.2, C171.2, C19.2, C215.2, C67.2, C78.2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; no longer C103.2, C134.2, C143.1, C145.1, C146.1, C149.2, C168.2, C174.2, C188.1, C190.+, C201.2, C39.2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
- net +3V3C: now also C125.2, C126.2, C127.2, C128.2, C129.2, C132.2, C133.2, C148.1, C158.1, C193.1, L2.2, R143.1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; no longer C179.2, C180.2, C181.2, C182.2, C183.2, C184.2, C189.1, C42.2, C96.1, C97.1, L7.2, R42.1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
- net +5V: now also C1.1, C114.2, C115.2, C120.+, C121.2, C122.2, C130.1, C131.+, C223.2, C225.+, C226.2, C227.+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; no longer C120.1, C121.+, C126.2, C128.+, C176.1, C2.2, C217.2, C3.+, C34.2, C46.+, C47.2, C48.+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
- net +5VA: now also C104.2, C105.+, C110.2, C15.2, C32.2, C53.2, C55.2, C76.2, C8.+, C90.2, C91.2, C92.2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; no longer C141.2, C160.2, C161.2, C162.+, C195.2, C198.2, C209.2, C68.2, C69.+, IC10P.V+, IC12P.V+, IC14P.V+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
- net A-A1: now also U15>NAME.PX33/EBI-ADDR[1]/SPI0-NPCS[3], U16.A0; no longer U1>NAME.PX33/EBI-ADDR[1]/SPI0-NPCS[3], U3.A0
- net A-A10: now also U15>NAME.PX24/EBI-ADDR[10]/EIM-SCAN[5], U16.A9; no longer U1>NAME.PX24/EBI-ADDR[10]/EIM-SCAN[5], U3.A9
- net A-A11: now also U15>NAME.PX23/EBI-ADDR[11]/EIM-SCAN[4], U16.A10; no longer U1>NAME.PX23/EBI-ADDR[11]/EIM-SCAN[4], U3.A10
- net A-A12: now also U15>NAME.PX22/EBI-ADDR[12]/EIM-SCAN[3]/TC-CLK2, U16.A11; no longer U1>NAME.PX22/EBI-ADDR[12]/EIM-SCAN[3]/TC-CLK2, U3.A11
- net A-A13: now also U15>NAME.PX21/EBI-ADDR[13]/EIM-SCAN[2]/TC-CLK1, U16.A12; no longer U1>NAME.PX21/EBI-ADDR[13]/EIM-SCAN[2]/TC-CLK1, U3.A12
- net A-A14: now also U15>NAME.PX20/EBI-ADDR[14]/EIM-SCAN[1]/TC-CLK0, U16.A13; no longer U1>NAME.PX20/EBI-ADDR[14]/EIM-SCAN[1]/TC-CLK0, U3.A13
- net A-A15: now also U15>NAME.PX19/EBI-ADDR[15]/EIM-SCAN[0]/TC-B2, U16.A14; no longer U1>NAME.PX19/EBI-ADDR[15]/EIM-SCAN[0]/TC-B2, U3.A14
- net A-A16: now also U15>NAME.PX18/EBI-ADDR[16]/TC-A2, U16.A15; no longer U1>NAME.PX18/EBI-ADDR[16]/TC-A2, U3.A15
- net A-A17: now also U15>NAME.PX17/EBI-ADDR[17]/TC-B1, U16.A16; no longer U1>NAME.PX17/EBI-ADDR[17]/TC-B1, U3.A16
- net A-A18: now also U15>NAME.PX16/EBI-ADDR[18]/USART3-CTS/TC-A1, U16.A17; no longer U1>NAME.PX16/EBI-ADDR[18]/USART3-CTS/TC-A1, U3.A17
- net A-A19: now also U15>NAME.PX15/EBI-ADDR[19]/USART3-RTS/TC-B0, U16.A18; no longer U1>NAME.PX15/EBI-ADDR[19]/USART3-RTS/TC-B0, U3.A18
- net A-A2: now also U15>NAME.PX32/EBI-ADDR[2]/SPI0-NPCS[2], U16.A1; no longer U1>NAME.PX32/EBI-ADDR[2]/SPI0-NPCS[2], U3.A1
- net A-A3: now also U15>NAME.PX31/EBI-ADDR[3]/SPI0-NPCS[1], U16.A2; no longer U1>NAME.PX31/EBI-ADDR[3]/SPI0-NPCS[1], U3.A2
- net A-A4: now also U15>NAME.PX30/EBI-ADDR[4]/SPI0-NPCS[0], U16.A3; no longer U1>NAME.PX30/EBI-ADDR[4]/SPI0-NPCS[0], U3.A3
- net A-A5: now also U15>NAME.PX29/EBI-ADDR[5]/SPI0-SCK, U16.A4; no longer U1>NAME.PX29/EBI-ADDR[5]/SPI0-SCK, U3.A4
- net A-A6: now also U15>NAME.PX28/EBI-ADDR[6]/SPI0-MOSI, U16.A5; no longer U1>NAME.PX28/EBI-ADDR[6]/SPI0-MOSI, U3.A5
- net A-A7: now also U15>NAME.PX27/EBI-ADDR[7]/SPI0-MISO, U16.A6; no longer U1>NAME.PX27/EBI-ADDR[7]/SPI0-MISO, U3.A6
- net A-A8: now also U15>NAME.PX26/EBI-ADDR[8]/EIM-SCAN[7], U16.A7; no longer U1>NAME.PX26/EBI-ADDR[8]/EIM-SCAN[7], U3.A7
- net A-A9: now also U15>NAME.PX25/EBI-ADDR[9]/EIM-SCAN[6], U16.A8; no longer U1>NAME.PX25/EBI-ADDR[9]/EIM-SCAN[6], U3.A8
- net A-D0: now also U15>NAME.PX10/EBI-DATA[0]/USART2-RXD, U16.IO0; no longer U1>NAME.PX10/EBI-DATA[0]/USART2-RXD, U3.IO0
- net A-D1: now also U15>NAME.PX09/EBI-DATA[1]/USART3-TXD, U16.IO1; no longer U1>NAME.PX09/EBI-DATA[1]/USART3-TXD, U3.IO1
- net A-D10: now also U15>NAME.PX00/EBI-DATA[10]/USART0-RXD, U16.IO10; no longer U1>NAME.PX00/EBI-DATA[10]/USART0-RXD, U3.IO10
- net A-D11: now also U15>NAME.PX39/EBI-DATA[11]/SPI1-NPCS[2], U16.IO11; no longer U1>NAME.PX39/EBI-DATA[11]/SPI1-NPCS[2], U3.IO11
- net A-D12: now also U15>NAME.PX38/EBI-DATA[12]/SPI1-NPCS[1], U16.IO12; no longer U1>NAME.PX38/EBI-DATA[12]/SPI1-NPCS[1], U3.IO12
- net A-D13: now also U15>NAME.PX37/EBI-DATA[13]/SPI1-NPCS[0], U16.IO13; no longer U1>NAME.PX37/EBI-DATA[13]/SPI1-NPCS[0], U3.IO13
- net A-D14: now also U15>NAME.PX36/EBI-DATA[14]/SPI1-SCK, U16.IO14; no longer U1>NAME.PX36/EBI-DATA[14]/SPI1-SCK, U3.IO14
- net A-D15: now also U15>NAME.PX35/EBI-DATA[15]/SPI1-MOSI, U16.A20/IO15; no longer U1>NAME.PX35/EBI-DATA[15]/SPI1-MOSI, U3.A20/IO15
- net A-D2: now also U15>NAME.PX08/EBI-DATA[2]/USART3-RXD, U16.IO2; no longer U1>NAME.PX08/EBI-DATA[2]/USART3-RXD, U3.IO2
- net A-D3: now also U15>NAME.PX07/EBI-DATA[3]/USART1-RTS, U16.IO3; no longer U1>NAME.PX07/EBI-DATA[3]/USART1-RTS, U3.IO3
- net A-D4: now also U15>NAME.PX06/EBI-DATA[4]/USART1-CTS, U16.IO4; no longer U1>NAME.PX06/EBI-DATA[4]/USART1-CTS, U3.IO4
- net A-D5: now also U15>NAME.PX05/EBI-DATA[5]/USART1-TXD, U16.IO5; no longer U1>NAME.PX05/EBI-DATA[5]/USART1-TXD, U3.IO5
- net A-D6: now also U15>NAME.PX04/EBI-DATA[6]/USART1-RXD, U16.IO6; no longer U1>NAME.PX04/EBI-DATA[6]/USART1-RXD, U3.IO6
- net A-D7: now also U15>NAME.PX03/EBI-DATA[7]/USART0-RTS, U16.IO7; no longer U1>NAME.PX03/EBI-DATA[7]/USART0-RTS, U3.IO7
- net A-D8: now also U15>NAME.PX02/EBI-DATA[8]/USART0-CTS, U16.IO8; no longer U1>NAME.PX02/EBI-DATA[8]/USART0-CTS, U3.IO8
- net A-D9: now also U15>NAME.PX01/EBI-DATA[9]/USART0-TXD, U16.IO9; no longer U1>NAME.PX01/EBI-DATA[9]/USART0-TXD, U3.IO9
- net A-RESET: now also C123.1, JP2.6, R159.1, U15>NAME.!RESET; no longer C1.1, JP1.6, R1.1, U1>NAME.!RESET
- net A-TCK: now also JP2.1, U15>NAME.TCK; no longer JP1.1, U1>NAME.TCK
- net A-TDI: now also JP2.9, U15>NAME.TDI; no longer JP1.9, U1>NAME.TDI
- net A-TDO: now also JP2.3, U15>NAME.TDO; no longer JP1.3, U1>NAME.TDO
- net A-TMS: now also JP2.5, U15>NAME.TMS; no longer JP1.5, U1>NAME.TMS
- net ABE0_: now also U23.DQML; no longer U9.DQML
- net ABE1_: now also U23.DQMH; no longer U9.DQMH
- net AD1939_RESET: now also R166.1, U17._PD/_RST; no longer R165.1, U14._PD/_RST
- net AGND: now also C105.-, C109.1, C11.2, C12.2, C130.2, C131.-, C14.-, C141.2, C15.1, C150.2, C16.2, C160.2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; no longer C100.-, C101.1, C102.-, C103.1, C105.2, C111.2, C113.1, C114.1, C117.1, C118.1, C120.2, C121.-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
- net B-A1: now also U23.A0; no longer U9.A0
- net B-A10: now also U23.A9; no longer U9.A9
- net B-A12: now also U23.A11; no longer U9.A11
- net B-A13: now also U23.A12; no longer U9.A12
- net B-A18: now also U23.BA0; no longer U9.BA0
- net B-A19: now also U23.BA1; no longer U9.BA1
- net B-A2: now also U23.A1; no longer U9.A1
- net B-A3: now also U23.A2; no longer U9.A2
- net B-A4: now also U23.A3; no longer U9.A3
- net B-A5: now also U23.A4; no longer U9.A4
- net B-A6: now also U23.A5; no longer U9.A5
- net B-A7: now also U23.A6; no longer U9.A6
- net B-A8: now also U23.A7; no longer U9.A7
- net B-A9: now also U23.A8; no longer U9.A8
- net B-D0: now also U23.DQ0; no longer U9.DQ0
- net B-D1: now also U23.DQ1; no longer U9.DQ1
- net B-D10: now also U23.DQ10; no longer U9.DQ10
- net B-D11: now also U23.DQ11; no longer U9.DQ11
- net B-D12: now also U23.DQ12; no longer U9.DQ12
- net B-D13: now also U23.DQ13; no longer U9.DQ13
- net B-D14: now also U23.DQ14; no longer U9.DQ14
- net B-D15: now also U23.DQ15; no longer U9.DQ15
- net B-D2: now also U23.DQ2; no longer U9.DQ2
- net B-D3: now also U23.DQ3; no longer U9.DQ3
- net B-D4: now also U23.DQ4; no longer U9.DQ4
- net B-D5: now also U23.DQ5; no longer U9.DQ5
- net B-D6: now also U23.DQ6; no longer U9.DQ6
- net B-D7: now also U23.DQ7; no longer U9.DQ7
- net B-D8: now also U23.DQ8; no longer U9.DQ8
- net B-D9: now also U23.DQ9; no longer U9.DQ9
- net B-HWAIT: now also R176.2, U15>NAME.PWM-PWM[4]/USART1-RXD/PA05; no longer R80.2, U1>NAME.PWM-PWM[4]/USART1-RXD/PA05
- net B-MISO: now also U15>NAME.USB-USB_ID/SPI0-MISO/PA11; no longer U1>NAME.USB-USB_ID/SPI0-MISO/PA11
- net B-MOSI: now also U15>NAME.USB-USB_VBOF/SPI0-MOSI/PA12; no longer U1>NAME.USB-USB_VBOF/SPI0-MOSI/PA12
- net B-RESET: now also U15>NAME.PWM-PWM[5]/USART1-TXD/PA06; no longer U1>NAME.PWM-PWM[5]/USART1-TXD/PA06
- net B-SCK: now also U15>NAME.SPI0-SCK/PA13; no longer U1>NAME.SPI0-SCK/PA13
- net B-SPISS: now also R173.1, U15>NAME.EIM-EXTINT[6]/SPI0-NPCS[0]/PA10; no longer R8.1, U1>NAME.EIM-EXTINT[6]/SPI0-NPCS[0]/PA10
- net BMODE0: now also R161.1; no longer R73.1
- net BMODE1: now also R162.1; no longer R72.1
- net CLKIN: now also R178.1; no longer R74.1
- net CLKOUT: now also R160.2; no longer R37.2
- net CS1: now also U15>NAME.PX14/EBI-NCS[1]/TC-A0, U16.!CE!; no longer U1>NAME.PX14/EBI-NCS[1]/TC-A0, U3.!CE!
- net CTS: now also U15>NAME.DAC-DATAN[0]/EIM-EXTINT[5]/USART0-CTS/PA04, U6.PB7(OC0A/OC1C/RTS); no longer U$8.PB7(OC0A/OC1C/RTS), U1>NAME.DAC-DATAN[0]/EIM-EXTINT[5]/USART0-CTS/PA04
- net CVOUT1: now also J20.6, U24.VOUTA; no longer J14.6, U17.VOUTA
- net CVOUT1^: now also IC1A.IN+, P10.6; no longer IC9A.IN+, P9.6
- net CVOUT2: now also J20.4, U24.VOUTB; no longer J14.4, U17.VOUTB
- net CVOUT2^: now also IC1B.IN+, P10.4; no longer IC9B.IN+, P9.4
- net CVOUT3: now also J20.5, U24.VOUTC; no longer J14.5, U17.VOUTC
- net CVOUT3^: now also IC1C.IN+, P10.5; no longer IC9C.IN+, P9.5
- net CVOUT4: now also J20.3, U24.VOUTD; no longer J14.3, U17.VOUTD
- net CVOUT4^: now also IC1D.IN+, P10.3; no longer IC9D.IN+, P9.3
- net DAC-LDAC: now also U24._LDAC; no longer U17._LDAC
- net DAC-RESET: now also U24._RESET; no longer U17._RESET
- net DM: now also J11.DM, R168.2; no longer J8.DM, R4.2
- net DP: now also J11.DP, R167.2; no longer J8.DP, R5.2
- net DR0PRI: now also U17.ASDATA1; no longer U14.ASDATA1
- net DR0SEC: now also U17.ASDATA2; no longer U14.ASDATA2
- net DT0PRI: now also U17.DSDATA1; no longer U14.DSDATA1
- net DT0SEC: now also U17.DSDATA2; no longer U14.DSDATA2
- net DT1SEC: now also U24.SDIN; no longer U17.SDIN
- net EMU_: now also R144.1; no longer R49.1
- net ENC0A: now also P8.7, U15>NAME.DAC-DATAN[0]/MACB-TXD[1]/PB03; no longer P1.7, U1>NAME.DAC-DATAN[0]/MACB-TXD[1]/PB03
- net ENC0A^: now also P9.13; no longer P2.13
- net ENC0B: now also P8.8, U15>NAME.DAC-DATA[0]/MACB-TXD[0]/PB02; no longer P1.8, U1>NAME.DAC-DATA[0]/MACB-TXD[0]/PB02
- net ENC0B^: now also P9.14; no longer P2.14
- net ENC1A: now also P8.5, U15>NAME.DAC-DATA[1]/MACB-RXD[0]/PB05; no longer P1.5, U1>NAME.DAC-DATA[1]/MACB-RXD[0]/PB05
- net ENC1A^: now also P9.11; no longer P2.11
- net ENC1B: now also P8.6, U15>NAME.EBI-NCS[3]/USART3-CLK/MACB-CRS/PB04; no longer P1.6, U1>NAME.EBI-NCS[3]/USART3-CLK/MACB-CRS/PB04
- net ENC1B^: now also P9.12; no longer P2.12
- net ENC2A: now also P8.3, U15>NAME.MACB-RX_ER/PB07; no longer P1.3, U1>NAME.MACB-RX_ER/PB07
- net ENC2A^: now also P9.9; no longer P2.9
- net ENC2B: now also P8.4, U15>NAME.DAC-DATAN[1]/MACB-RXD[1]/PB06; no longer P1.4, U1>NAME.DAC-DATAN[1]/MACB-RXD[1]/PB06
- net ENC2B^: now also P9.10; no longer P2.10
- net ENC3A: now also P8.1, U15>NAME.MACB-MDIO/PB09; no longer P1.1, U1>NAME.MACB-MDIO/PB09
- net ENC3A^: now also P9.7; no longer P2.7
- net ENC3B: now also P8.2, U15>NAME.MACB-MDC/PB08; no longer P1.2, U1>NAME.MACB-MDC/PB08
- net ENC3B^: now also P9.8; no longer P2.8
- net GAINL-1: now also C54.+, C59.1, IC6B.OUT, J10._0; no longer IC14B.IN-, J13._0, R182.2
- net GAINL-2: now also C59.2, IC6B.IN-, R12.1, R14.1, R79.2; no longer C208.+, IC14B.OUT
- net GAINR-1: now also C56.+, C60.1, IC7B.OUT, J10.0; no longer IC13B.IN-, J13.0, R175.2
- net GAINR-2: now also C60.2, IC7B.IN-, R5.1, R80.2, R9.1; no longer C197.+, IC13B.OUT
- net GND: now also C10.-, C111.2, C112.1, C113.1, C114.1, C115.1, C116.1, C117.1, C118.1, C119.1, C120.-, C121.1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; no longer C10.2, C11.2, C12.2, C127.-, C128.-, C13.2, C14.2, C15.2, C16.2, C17.2, C176.2, C179.1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
- net HBE: now also U15>NAME.PX11/EBI-NWE1/USART2-TXD, U16.!BHE!; no longer U1>NAME.PX11/EBI-NWE1/USART2-TXD, U3.!BHE!
- net HPL: now also IC5B.IN+, P6.1; no longer IC15B.IN+, P3.1
- net HPL-J: now also C9.+, J1.R; no longer C165.+, J3.R
- net HPL^: now also P2.4, P7.1; no longer P4.1, P6.4
- net HPR: now also IC5A.IN+, P6.3; no longer IC15A.IN+, P3.3
- net HPR-J: now also C7.-, J1.T; no longer C164.-, J3.T
- net HPR^: now also P2.1, P7.3; no longer P4.3, P6.1
- net IN-VREF: now also IC13A.IN-, IC13A.OUT, P4.2, P4.3, P5.2, P5.3, R77.1, R78.1, R79.1, R80.1; no longer IC12A.IN-, IC12A.OUT, P7.2, P7.3, P8.2, P8.3, R176.1, R177.1, R183.1, R184.1
- net IN1L: now also L9.2, P6.9; no longer L3.2, P3.9
- net IN1L+: now also C170.2, C174.2, R171.1, U17.ADC1LP; no longer C153.2, C154.2, R139.1, U14.ADC1LP
- net IN1L-: now also C174.1, C180.1, R172.1, U17.ADC1LN; no longer C152.1, C154.1, R135.1, U14.ADC1LN
- net IN1L-J: now also C11.1, P6.10, R16.2; no longer J4.TT, P3.10
- net IN1L-J^: now also C57.-, P7.10; no longer C211.-, P4.10
- net IN1L^: now also C54.-, D11.A, P7.9, R120.2, R73.2, U19A.+IN; no longer C208.-, P4.9, R185.2
- net IN1R: now also L10.2, P6.11; no longer L4.2, P3.11
- net IN1R+: now also C134.2, C135.2, R163.1, U17.ADC1RP; no longer C138.2, C139.2, R115.1, U14.ADC1RP
- net IN1R-: now also C135.1, C141.1, R164.1, U17.ADC1RN; no longer C137.1, C139.1, R112.1, U14.ADC1RN
- net IN1R-J: now also C12.1, P6.12, R20.2; no longer J5.TT, P3.12
- net IN1R-J^: now also C58.-, P7.12; no longer C196.-, P4.12
- net IN1R^: now also C56.-, D12.A, P7.11, R121.2, R74.2, U20A.+IN; no longer C197.-, P4.11, R178.2
- net IN2-L: now also J4.TT, L6.2; no longer J11.TT, L5.2
- net IN2-R: now also J5.TT, L7.2; no longer J12.TT, L6.2
- net IN2L+: now also C217.2, C221.2, R185.1, U17.ADC2LP; no longer C172.2, C173.2, R144.1, U14.ADC2LP
- net IN2L-: now also C214.1, C217.1, R183.1, U17.ADC2LN; no longer C171.1, C173.1, R141.1, U14.ADC2LN
- net IN2R+: now also C216.2, C220.2, R184.1, U17.ADC2RP; no longer C205.2, C206.2, R173.1, U14.ADC2RP
- net IN2R-: now also C213.1, C216.1, R182.1, U17.ADC2RN; no longer C204.1, C206.1, R170.1, U14.ADC2RN
- net KEY0: now also P8.12, U15>NAME.EBI-NCS[0]/EIM-SCAN[0]/ADC-AD[4]/PA25; no longer P1.12, U1>NAME.EBI-NCS[0]/EIM-SCAN[0]/ADC-AD[4]/PA25
- net KEY0^: now also P9.18, U25C.O; no longer P2.18, U19C.O
- net KEY1: now also P8.11, U15>NAME.EBI-ADDR[20]/EIM-SCAN[1]/ADC-AD[5]/PA26; no longer P1.11, U1>NAME.EBI-ADDR[20]/EIM-SCAN[1]/ADC-AD[5]/PA26
- net KEY1^: now also P9.17, U25B.O; no longer P2.17, U19B.O
- net KEY2: now also P8.10, U15>NAME.EBI-ADDR[21]/EIM-SCAN[2]/ADC-AD[6]/PA27; no longer P1.10, U1>NAME.EBI-ADDR[21]/EIM-SCAN[2]/ADC-AD[6]/PA27
- net KEY2^: now also P9.16, U25A.O; no longer P2.16, U19A.O
- net KEY3: now also P8.9, U15>NAME.EBI-ADDR[22]/EIM-SCAN[3]/ADC-AD[7]/PA28; no longer P1.9, U1>NAME.EBI-ADDR[22]/EIM-SCAN[3]/ADC-AD[7]/PA28
- net KEY3^: now also P9.15, U25D.O; no longer P2.15, U19D.O
- net LBE: now also U15>NAME.PX34/EBI-ADDR[0]/SPI1-MISO, U16.!BLE!; no longer U1>NAME.PX34/EBI-ADDR[0]/SPI1-MISO, U3.!BLE!
- net MMC-DETECT: now also R134.1, U15>NAME.USART3-RTS/USART2-RTS/MACB-TX_CLK/PB00; no longer R13.1, U1>NAME.USART3-RTS/USART2-RTS/MACB-TX_CLK/PB00
- net MMC-PROTECT: now also R137.1, U15>NAME.USART3-CTS/USART2-CTS/MACB-TX_EN/PB01; no longer R14.1, U1>NAME.USART3-CTS/USART2-CTS/MACB-TX_EN/PB01
- net MODE-KEY: now also P8.13, U15>NAME.DAC-DATAN[1]/EIM-EXTINT[3]/ADC-AD[3]/PA24; no longer P1.13, U1>NAME.DAC-DATAN[1]/EIM-EXTINT[3]/ADC-AD[3]/PA24
- net MODE-KEY^: now also P9.19, U25E.O; no longer P2.19, U19E.O
- net MODE-LED: now also P8.14, U15>NAME.DAC-DATA[1]/EIM-EXTINT[2]/ADC-AD[2]/PA23; no longer P1.14, U1>NAME.DAC-DATA[1]/EIM-EXTINT[2]/ADC-AD[2]/PA23
- net MODE-LED^: now also P9.20, R61.1; no longer P2.20, R21.1
- net N$1: now also IC1A.IN-, R1.2, R3.1; no longer IC9A.IN-, R146.1, R147.2
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
Commit message: spreadsheets and eagle
Parts:
- added P12: M-1X03-SIP-100-40, con-headers-jp:M-1X03-SIP-100-40
- C27: device rc-master-smd:C_1206 -> rc-master-smd:C_0603
- C28: device rc-master-smd:CP_3528 -> rc-master-smd:CP_1206/T
- C29, C30: value 12p -> 8p
- IC11, IC13, IC5, IC6, IC7, IC8: value AD8607R -> AD8606
- L10, L2, L3, L5, L6, L7, L9: device rc-master-smd:L_1206 -> rc-master-smd:L_0603
Connections:
- new net N$155: DSP1.TX, P12.3
- new net N$183: DSP1.RX, P12.2
- net GND: now also P12.1

Commit message: final circuit
Parts:
- R187: value 47k -> 18k
- R188: value 330k -> 47k
- R192: value 117k -> 118k
- R45: value 3.32k -> 3k32
Changed lines of the file:
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@@
 <part name="R40" library="rc-master-smd" deviceset="R_" device="0603" value="0"/>
 <part name="J9" library="monome-inc" deviceset="PHA2U" device=""/>
-<part name="R188" library="rc-master-smd" deviceset="R_" device="0603" value="330k"/>
-<part name="R187" library="rc-master-smd" deviceset="R_" device="0603" value="47k"/>
+<part name="R188" library="rc-master-smd" deviceset="R_" device="0603" value="47k"/>
+<part name="R187" library="rc-master-smd" deviceset="R_" device="0603" value="18k"/>
 <part name="GND46" library="supply" deviceset="GND" device=""/>
 <part name="GND1" library="supply" deviceset="GND" device=""/>
@@
 <part name="L8" library="inductor-bourns" deviceset="SRR6038" device="" value="SRR6038-100Y"/>
 <part name="R72" library="rc-master-smd" deviceset="R_" device="0603" value="0"/>
-<part name="R45" library="rc-master-smd" deviceset="R_" device="0603" value="3.32k"/>
+<part name="R45" library="rc-master-smd" deviceset="R_" device="0603" value="3k32"/>
 <part name="GND50" library="supply" deviceset="GND" device=""/>
 <part name="GND51" library="supply" deviceset="GND" device=""/>
@@
 <part name="L1" library="monome-inc" deviceset="XAL7030-103" device=""/>
 <part name="C10" library="rc-master-smd" deviceset="CP_" device="1206/T" value="4.7u"/>
-<part name="R192" library="rc-master-smd" deviceset="R_" device="0603" value="117k"/>
+<part name="R192" library="rc-master-smd" deviceset="R_" device="0603" value="118k"/>
 <part name="R194" library="rc-master-smd" deviceset="R_" device="0603" value="13k3"/>
 <part name="C1" library="rc-master-smd" deviceset="C_" device="1206" value="2.2u"/>

Commit message: circuits and mechanicals
Parts:
- removed LED9: (no value), led:LEDCHIPLED_0805
- removed R108: 10k, rc-master-smd:R_0603
- added C229: 100u, rc-master-smd:CP_7343-43
- C218: device rc-master-smd:CP_1206/T -> rc-master-smd:CP_6032-28
- C222: value 470n -> 100n
- C28: value 47u -> 100u; device rc-master-smd:CP_1206/T -> rc-master-smd:CP_7343-43
- J1, J21, J22: value STEREOSW2GND -> STEREOSW3GND; device Audio Jacks 0.25 inch:STEREOSW2GND -> monome-inc:STEREOSW3GND
- J8: device con-cuistack:PJ-102AH/BH -> monome-inc:PJ-102AH/BH
- LED12, LED8: device led:LEDCHIPLED_1206 -> led:LEDCHIPLED_0805
- R119, R120, R121: value 470k -> 47k
Connections:
- removed net N$199: LED9.A, R108.1, U18A.-IN
- new net A-INT: DSP1.PF12, U15>NAME.EIM-SCAN[6]/PM-GCLK[2]/PWM-PWM[2]/PB21
- new net B-INT: DSP1.PF13, U15>NAME.EIM-SCAN[5]/PM-GCLK[1]/PWM-PWM[1]/PB20
- net +12V: now also P8.2; no longer P8.24
- net +3V3: now also P8.3; no longer P8.25
- net +5V: now also C229.+, P8.4; no longer P8.26
- net +5VA: no longer R108.2
- net AGND: now also J1.SN, U18A.+IN; no longer J1.S, LED9.C
- net ENC0A: now also P8.13; no longer P8.7
- net ENC0B: now also P8.14; no longer P8.8
- net ENC1A: now also P8.11; no longer P8.5
- net ENC1B: now also P8.12; no longer P8.6
- net ENC2A: now also P8.9; no longer P8.3
- net ENC2B: now also P8.10; no longer P8.4
- net ENC3A: now also P8.7; no longer P8.1
- net ENC3B: now also P8.8; no longer P8.2
- net GND: now also C229.-, J21.SN, J22.SN, P8.1, P8.5, P8.6; no longer J21.S, J22.S, P8.23, P8.27, P8.28
- net HPL-J: now also C9.-; no longer C9.+
- net KEY0: now also P8.18; no longer P8.12
- net KEY1: now also P8.17; no longer P8.11
- net KEY2: now also P8.16; no longer P8.10
- net KEY3: now also P8.15; no longer P8.9
- net MODE-KEY: now also P8.19; no longer P8.13
- net MODE-LED: now also P8.20; no longer P8.14
- net N$154: now also C9.+; no longer C9.-
- net N$195: now also U18A.-IN; no longer U18A.+IN
- net OLED-DC: now also P8.21; no longer P8.15
- net OLED-RES: now also P8.22; no longer P8.16
- net SPI1-CS0: now also P8.23; no longer P8.17
- net SPI1-CS1: now also P8.24; no longer P8.18
- net SPI1-MISO: now also P8.26; no longer P8.20
- net SPI1-MOSI: now also P8.27; no longer P8.21
- net SPI1-SCK: now also P8.28; no longer P8.22
Other:
- moved on the sheet: C114, C120, C68, C70, C9, U18A

Commit message: final circuit build notes
Parts:
- removed LED10, LED11: (no value), led:LEDCHIPLED_0805
- removed R109, R110: 10k, rc-master-smd:R_0603
- removed U18, U19, U20: TL072D, linear:TL072D
- added IC14, IC15: AD8606, analog-devices:AD8607R
- added IC16: AD8607R, analog-devices:AD8607R
Connections:
- removed net N$168: LED10.A, R109.1, U19A.-IN
- removed net N$174: LED5.A, R58.2
- removed net N$181: C58.+, IC7A.IN-
- removed net N$187: LED11.A, R110.1, U20A.-IN
- removed net N$189: LED7.A, R60.2
- net +5VA: now also IC14P.V+, IC15P.V+, IC16P.V-, LED7.A; no longer R109.2, R110.2, U18P.V+, U19P.V+, U20P.V+
- net AGND: now also IC14A.IN+, IC14P.V-, IC15A.IN+, IC15P.V-, IC16A.IN+, IC16B.IN+, IC16B.IN-, IC16P.V+; no longer LED10.C, LED11.C, LED5.C, LED7.C, U18A.+IN, U18B.+IN, U18B.-IN, U18P.V-, U19P.V-, U20P.V-
- net IN1L^: now also IC15A.IN-; no longer U19A.+IN
- net IN1R^: now also IC14A.IN-; no longer U20A.+IN
- net N$153: now also C57.+
- net N$158: now also IC6A.IN-
- net N$162: now also IC15A.OUT; no longer U19A.OUT
- net N$164: now also LED7.C, R60.2; no longer C57.+, IC6A.IN-
- net N$167: now also IC15B.IN-; no longer U19B.-IN
- net N$169: now also C58.+
- net N$172: now also IC7A.IN-
- net N$178: now also IC15B.OUT; no longer U19B.OUT
- net N$179: now also IC15B.IN+; no longer U19B.+IN
- net N$184: now also IC14A.OUT; no longer U20A.OUT
- net N$186: now also IC14B.IN-; no longer U20B.-IN
- net N$190: now also IC14B.OUT; no longer U20B.OUT
- net N$191: now also IC14B.IN+; no longer U20B.+IN
- net N$195: now also IC16A.IN-; no longer U18A.-IN
- net N$196: now also IC16A.OUT; no longer U18A.OUT
Other:
- moved on the sheet: C57, C58, LED5, LED7, R58, R60

Commit message: notes from sept proto build;
Connections:
- net N$120 renamed U-MOSI
- net N$121 renamed U-SCK
- net N$14 renamed U-MISO
Changed lines of the file:
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@@
 </segment>
 </net>
-<net name="N$14" class="0">
+<net name="U-MISO" class="0">
 <segment>
 <pinref part="P1" gate="G$1" pin="2"/>
@@
 </segment>
 </net>
-<net name="N$120" class="0">
+<net name="U-MOSI" class="0">
 <segment>
 <pinref part="P1" gate="G$1" pin="3"/>
@@
 </segment>
 </net>
-<net name="N$121" class="0">
+<net name="U-SCK" class="0">
 <segment>
 <pinref part="P1" gate="G$1" pin="4"/>
