File: circuit/aleph-dev/aleph.sch (EAGLE design)
At the start: 571 parts, among them IC1 AD8567, IC10 AD8606, IC11 AD8606, IC12 AD8606, IC13 AD8606, IC14 AD8606, IC15 AD8606, IC16 AD8607R, IC2 AD8606, IC3 AD8606, IC4 AD8606, IC5 AD8606, IC6 AD8606, IC7 AD8606, IC8 AD8606, IC9 AD8606, J1 STEREOSW3GND, J10 PHA2U, J11 USBA-VERT, J12 STX-3680, J13 STX-3680, J14 STX-3680, J15 STX-3680, J16 STX-3680, J17 STX-3680, J18 STX-3680, J19 STX-3680, J2 NSJ12HF, J20 F-2X03-DIL-100, J21 STEREOSW3GND, J22 STEREOSW3GND, J3 NSJ12HF, J4 NSJ12HF, J5 NSJ12HF, J6 SJ1-3533NG, J8 PJ-102AH/BH, J9 PHA2U, K1 PVA1, K2 PVA1, K3 PVA1, K4 PVA1, P1 M-1X05-SIP-100-32, P10 M-2X03-DIL-100, P12 M-1X03-SIP-100-40, P2 EVJ-POT, P3 EVJ-POT, P4 EVJ-POT, P5 EVJ-POT, P6 F-2X06-DIL-100, P7 M-2X06-DIL-100, P8 M-2X14-DIL-100, P9 M-2X14-DIL-100, SW1 PANASONIC-EVQ, U1 BAS70-04, U10 FDS9431A, U11 BAS70-04, U12 BAS70-04, U13 BAS70-04, U14 BAS70-04, U15 AT32UC3A0512, U16 CY62167EV30-Z, U17 AD1939, U2 LMR62014, U21 AD7923, U22 LM4040M3, U23 MT48LC32M16A2tg-75, U24 AD5686R, U25 74HC14D, U26 SN74LVC2G14, U3 BAS70-04, U4 TPS2020, U5 LM2678, U6 ATMEGA32U4-AU, U7 ADP3339, U8 TPA6111A2, U9 ADP3339, X1 16mhz, Y1 ASFL1-27mhz, Y2 12mhz, Y3 ASFL1-12.288mhz

Commit message: after seattle
Parts:
- IC16: value AD8607R -> AD8606
Connections:
- new net N$168: LED5.C, R58.2
- net +5VA: now also IC16P.V+, LED5.A; no longer IC16P.V-
- net AGND: now also IC16P.V-; no longer IC16P.V+
Other:
- moved on the sheet: IC16P
Changed lines of the file:
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@@
 <setting verticaltext="up"/>
 </settings>
-<grid distance="0.1" unitdist="inch" unit="inch" style="lines" multiple="1" display="no" altdistance="0.01" altunitdist="inch" altunit="inch"/>
+<grid distance="0.05" unitdist="inch" unit="inch" style="lines" multiple="1" display="no" altdistance="0.01" altunitdist="inch" altunit="inch"/>
 <layers>
 <layer number="1" name="Top" color="4" fill="1" visible="no" active="no"/>
@@
 <part name="V88" library="supply" deviceset="+5VA" device=""/>
 <part name="V92" library="supply" deviceset="+5VA" device=""/>
-<part name="IC16" library="analog-devices" deviceset="AD8607" device="R"/>
+<part name="IC16" library="analog-devices" deviceset="AD8607" device="R" value="AD8606"/>
 </parts>
 <sheets>
@@
 <instance part="IC16" gate="A" x="217.17" y="306.07" rot="MR180"/>
 <instance part="IC16" gate="B" x="281.94" y="330.2" rot="MR180"/>
-<instance part="IC16" gate="P" x="322.58" y="308.61" rot="MR180"/>
+<instance part="IC16" gate="P" x="322.58" y="308.61" rot="MR0"/>
 </instances>
 <busses>
@@
 <pinref part="AGND91" gate="VR1" pin="AGND"/>
 <wire x1="322.58" y1="298.45" x2="322.58" y2="299.72" width="0.1524" layer="91"/>
+<pinref part="IC16" gate="P" pin="V-"/>
 <wire x1="322.58" y1="299.72" x2="322.58" y2="300.99" width="0.1524" layer="91"/>
 <junction x="322.58" y="299.72"/>
-<pinref part="IC16" gate="P" pin="V+"/>
 </segment>
 <segment>
@@
 <wire x1="322.58" y1="317.5" x2="316.23" y2="317.5" width="0.1524" layer="91"/>
 <wire x1="316.23" y1="317.5" x2="316.23" y2="311.15" width="0.1524" layer="91"/>
-<wire x1="322.58" y1="316.23" x2="322.58" y2="317.5" width="0.1524" layer="91"/>
 <pinref part="V95" gate="G$1" pin="+5VA"/>
 <wire x1="322.58" y1="317.5" x2="322.58" y2="318.77" width="0.1524" layer="91"/>
+<pinref part="IC16" gate="P" pin="V+"/>
+<wire x1="322.58" y1="316.23" x2="322.58" y2="317.5" width="0.1524" layer="91"/>
 <junction x="322.58" y="317.5"/>
-<pinref part="IC16" gate="P" pin="V-"/>
 </segment>
 </net>
@@
 <wire x1="138.43" y1="196.85" x2="138.43" y2="198.12" width="0.1524" layer="91"/>
 </segment>
+<segment>
+<pinref part="LED5" gate="G$1" pin="A"/>
+<pinref part="V92" gate="G$1" pin="+5VA"/>
+<wire x1="138.43" y1="62.23" x2="138.43" y2="63.5" width="0.1524" layer="91"/>
+</segment>
 </net>
 <net name="N$165" class="0">
@@
 </segment>
 </net>
+<net name="N$168" class="0">
+<segment>
+<pinref part="R58" gate="G$1" pin="2"/>
+<pinref part="LED5" gate="G$1" pin="C"/>
+<wire x1="138.43" y1="53.34" x2="138.43" y2="54.61" width="0.1524" layer="91"/>
+</segment>
+</net>
