File: circuit/aleph-dev/aleph.brd (EAGLE design)
At the start: 370.8 x 111.8 mm, 477 parts, among them IC1 AD8606, IC2 AD8606, IC3 AD8606, IC4 AD8606, IC5 AD8606, IC6 AD8606, IC7 AD8607R, IC8 AD8606, IC9 AD8567, J1 SJ1-3533NG, J10 PHA2U, J11 NSJ12HF, J12 NSJ12HF, J15 STX-3680, J16 STX-3680, J17 STX-3680, J18 STX-3680, J19 STX-3680, J2 PJ-102AH/BH, J20 STX-3680, J21 STX-3680, J22 STX-3680, J3 STEREOSW2GND, J4 NSJ12HF, J5 NSJ12HF, J6 STEREOSW2GND, J7 STEREOSW2GND, J8 USBA-VERT, K0 PVA1, K1 PVA1, K2 PVA1, K3 PVA1, P1 M-2X14-DIL-100, P2 M-2X14-DIL-100, P3 M-2X09-DIL-100, P4 M-2X09-DIL-100, P5 EVJ-POT, P6 EVJ-POT, P7 EVJ-POT, P8 EVJ-POT, U1 AT32UC3A0512, U10 LM4040M3, U14 AD1939, U17 AD5686R, U18 FDS9431A, U19 74HC14D, U2 FT232RL, U20 SN74LVC2G14, U21 LM2674, U22 BAS70-04, U23 BAS70-04, U24 BAS70-04, U25 BAS70-04, U3 CY62167EV30-Z, U4 TPS2020, U5 AD7923, U6 LM2678, U7 ADP3339, U8 ADP3339, U9 MT48LC32M16A2tg-75, Y1 12mhz, Y2 ASFL1-27mhz, Y3 ASFL1-12.288mhz

Commit message: march 2013 build
Parts:
- removed R166: 100k, rc-master-smd:R0603
- C18: device rc-master-smd:C0603 -> rc-master-smd:C1206
- C43: device rc-master-smd:C1206 -> rc-master-smd:C1206/T
- C46: device rc-master-smd:C3225 -> rc-master-smd:C3528/T
- C75: device rc-master-smd:C3528/T -> rc-master-smd:C1210/T
- R36: value 100k -> 10k
- R64: value 100k -> 47k
- moved C18 5.36 mm to (136.7, 68.1), turned to 90 degrees
- moved C13 2.54 mm to (139.1, 67.3)
- moved C9 2.54 mm to (141.0, 67.3)
- moved C17 0.95 mm to (132.7, 66.7)
Connections:
- net +3V3: now also U3.47
- net +3V3C: now also U14.31; no longer R166.1
- net +5V: now also C46.-; no longer C46.1
- net B-MISO: no longer U14.31
- net B-MOSI: no longer U14.30
- net B-SCK: no longer U14.34
- net B-SPISEL4: no longer R166.2, U14.35
- net GND: now also C43.-, C46.+, U14.30, U14.34, U14.35; no longer C43.1, C46.2, U3.47
- net UNREG_IN: now also C43.+; no longer C43.2
Routing:
- net B-SPISEL4: track 18.2 -> 0.00 mm, vias 1 -> 0
- net B-SCK: track 61.6 -> 46.0 mm, vias 3 -> 2
- net B-MISO: track 62.4 -> 48.5 mm, vias 3 -> 2
- net B-MOSI: track 61.9 -> 48.5 mm, vias 3 -> 2
- net GND: track 473.2 -> 483.8 mm
- net +3V3: track 411.6 -> 418.2 mm, vias 14 -> 15
- net VDDOUT: track 17.7 -> 20.7 mm
- net VDDIO: track 42.8 -> 40.3 mm
- net DT1SEC: track 34.4 -> 32.7 mm
- net +3V3C: track 134.4 -> 134.8 mm, vias 20 -> 19
Other:
- board text added: "130315"
- board text added: "SS"
- board text removed: "SEL4"

Commit message: arrived
Parts:
- removed C140: 100n, rc-master-smd:C0603
- removed C141, C160: 330p, rc-master-smd:C0603
- removed C155, C161: 680p, rc-master-smd:C0603
- removed C156, C162: 100p, rc-master-smd:C0603
- removed C157, C163: 220p, rc-master-smd:C0603
- removed C158, C164: 2200p, rc-master-smd:C0603
- removed C159, C165: 10u, rc-master-smd:C1206/T
- removed IC4: AD8606, analog-devices:SO8
- removed R117, R124: 11k, rc-master-smd:R0603
- removed R118, R120, R125, R127: 5k49, rc-master-smd:R0603
- removed R119, R126: 3k32, rc-master-smd:R0603
- removed R121, R128: 604, rc-master-smd:R0603
- removed R122, R129: 1k65, rc-master-smd:R0603
- removed R123, R130: 49k9, rc-master-smd:R0603
- removed R131, R132: 2k74, rc-master-smd:R0603
Connections:
- removed net N$102: C141.2, R117.1, R119.2, R120.2
- removed net N$103: C155.1, R118.1, R122.1, R131.1
- removed net N$107: C157.2, IC4.3, R122.2
- removed net N$109: C156.2, IC4.1, R120.1, R121.1
- removed net N$111: C158.2, C159.+, R121.2
- removed net N$112: C156.1, IC4.2, R119.1
- removed net N$113: C160.2, R124.1, R126.2, R127.2
- removed net N$114: C161.1, R125.1, R129.1, R132.1
- removed net N$115: C163.2, IC4.5, R129.2
- removed net N$120: C162.2, IC4.7, R127.1, R128.1
- removed net N$121: C164.2, C165.+, R128.2
- removed net N$122: C162.1, IC4.6, R126.1
- net +3V3A: no longer C140.2, IC4.8
- net +5V: now also C46.+; no longer C46.-
- net AGND: no longer C140.1, C141.1, C155.2, C157.1, C158.1, C160.1, C161.2, C163.1, C164.1, IC4.4, R123.2, R130.2
- net GND: now also C46.-; no longer C46.+
- net HP-LP: no longer C165.-, R130.1
- net HP-RP: no longer C159.-, R123.1
- net HPL+: no longer R125.2
- net HPL-: no longer R124.2
- net HPR+: no longer R118.2
- net HPR-: no longer R117.2
- net VREF: no longer R131.2, R132.2
Routing:
- net HPL-: track 39.2 -> 0.00 mm, vias 2 -> 0
- net HP-RP: track 38.6 -> 0.00 mm, vias 2 -> 0
- net HPL+: track 37.3 -> 0.00 mm
- net HPR-: track 35.0 -> 0.00 mm
- net VREF: track 244.8 -> 210.5 mm, vias 9 -> 7
- net HPR+: track 31.8 -> 0.00 mm
- net HP-LP: track 29.0 -> 0.00 mm, vias 2 -> 0
- net AGND: track 241.7 -> 213.8 mm, vias 53 -> 48
- net IN1R+: track 54.9 -> 45.9 mm
- net IN1R-: track 53.9 -> 45.7 mm
- net N$120: track 7.20 -> 0.00 mm
- net N$103: track 6.60 -> 0.00 mm
- net N$114: track 6.60 -> 0.00 mm
- net N$109: track 6.37 -> 0.00 mm
- net N$121: track 6.36 -> 0.00 mm, vias 1 -> 0
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
Commit message: cleanup
Routing:
- net +5VA: track 232.6 -> 179.3 mm, vias 2 -> 8
- net N$34: track 15.4 -> 22.8 mm
- net N$52: track 15.4 -> 22.8 mm
- net N$48: track 15.4 -> 22.8 mm
- net N$42: track 15.4 -> 22.8 mm
- net N$51: track 6.60 -> 10.3 mm
- net N$41: track 6.60 -> 10.3 mm
- net N$33: track 6.60 -> 10.3 mm
- net N$47: track 6.60 -> 10.3 mm
- net N$56: track 28.9 -> 32.4 mm
- net N$138: track 48.9 -> 52.4 mm
- net N$139: track 17.2 -> 20.6 mm
- net N$137: track 78.5 -> 81.9 mm
- net CVOUT4^: track 217.4 -> 218.3 mm
- net CVOUT3^: track 210.9 -> 211.6 mm
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
Commit message: todos
Parts:
- R162: value 100k -> 1k
Routing:
- net +5VA: track 179.3 -> 187.1 mm
- net +3V3: track 418.2 -> 422.4 mm
Changed lines of the file:
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@@
 <attribute name="VALUE" x="36.5125" y="22.86" size="1.016" layer="28" font="vector" ratio="12" rot="MR180"/>
 </element>
-<element name="R162" library="rc-master-smd" package="R0603" value="100k" x="162.56" y="97.155" smashed="yes" rot="MR270">
+<element name="R162" library="rc-master-smd" package="R0603" value="1k" x="162.56" y="97.155" smashed="yes" rot="MR270">
 <attribute name="NAME" x="161.925" y="99.06" size="1.016" layer="26" font="vector" ratio="12" rot="MR90"/>
 <attribute name="VALUE" x="164.465" y="98.425" size="1.016" layer="28" font="vector" ratio="12" rot="MR270"/>
@@
 <wire x1="279.4" y1="43.815" x2="279.4" y2="44.323" width="0.254" layer="1"/>
 <wire x1="279.4" y1="44.323" x2="279.527" y2="44.45" width="0.254" layer="1"/>
-<wire x1="280.035" y1="46.99" x2="283.21" y2="46.99" width="0.4064" layer="1"/>
-<via x="283.21" y="46.99" extent="1-16" drill="0.381"/>
-<wire x1="283.21" y1="46.99" x2="292.735" y2="46.99" width="0.4064" layer="16"/>
-<wire x1="292.735" y1="46.99" x2="295.91" y2="46.99" width="0.4064" layer="1"/>
+<wire x1="280.035" y1="46.99" x2="283.845" y2="46.99" width="0.4064" layer="1"/>
+<wire x1="283.845" y1="46.99" x2="288.925" y2="52.07" width="0.4064" layer="1"/>
+<via x="288.925" y="52.07" extent="1-16" drill="0.381"/>
+<wire x1="288.925" y1="52.07" x2="294.005" y2="46.99" width="0.4064" layer="16"/>
+<wire x1="294.005" y1="46.99" x2="295.91" y2="46.99" width="0.4064" layer="1"/>
 <wire x1="295.91" y1="46.99" x2="304.8" y2="55.88" width="0.4064" layer="1"/>
 <wire x1="304.8" y1="55.88" x2="341.15" y2="55.88" width="0.4064" layer="1"/>
 <wire x1="341.15" y1="55.88" x2="353.85" y2="68.58" width="0.4064" layer="1"/>
-<via x="292.735" y="46.99" extent="1-16" drill="0.381"/>
+<via x="294.005" y="46.99" extent="1-16" drill="0.381"/>
 <wire x1="222.25" y1="17.145" x2="222.25" y2="16.51" width="0.6096" layer="1"/>
 <wire x1="222.25" y1="16.51" x2="219.71" y2="13.97" width="0.6096" layer="1"/>
@@
 <wire x1="285.75" y1="43.18" x2="289.56" y2="43.18" width="0.4064" layer="1"/>
 <wire x1="289.56" y1="43.18" x2="289.56" y2="36.195" width="0.4064" layer="1"/>
-<wire x1="289.56" y1="43.18" x2="292.1" y2="43.18" width="0.4064" layer="1"/>
-<via x="292.1" y="43.18" extent="1-16" drill="0.381"/>
-<wire x1="292.1" y1="43.18" x2="294.64" y2="45.72" width="0.4064" layer="16"/>
-<wire x1="294.64" y1="45.72" x2="294.64" y2="49.53" width="0.4064" layer="16"/>
 <wire x1="364.4265" y1="83.8835" x2="363.22" y2="85.09" width="0.4064" layer="1"/>
 <contactref element="L10" pad="1"/>
@@
 <wire x1="317.5" y1="57.785" x2="304.8" y2="57.785" width="0.4064" layer="1"/>
 <wire x1="304.8" y1="57.785" x2="302.895" y2="57.785" width="0.4064" layer="1"/>
-<wire x1="302.895" y1="57.785" x2="294.64" y2="49.53" width="0.4064" layer="1"/>
-<via x="294.64" y="49.53" extent="1-16" drill="0.381"/>
+<wire x1="302.895" y1="57.785" x2="300.99" y2="55.88" width="0.4064" layer="1"/>
 <via x="304.8" y="57.785" extent="1-16" drill="0.381"/>
 <via x="317.5" y="57.785" extent="1-16" drill="0.381"/>
 <via x="330.2" y="57.785" extent="1-16" drill="0.381"/>
+<wire x1="300.99" y1="55.88" x2="289.56" y2="44.45" width="0.4064" layer="1"/>
 <wire x1="304.8" y1="57.785" x2="304.8" y2="64.77" width="0.254" layer="16"/>
 <via x="304.8" y="64.77" extent="1-16" drill="0.381"/>
@@
 <wire x1="317.5" y1="57.785" x2="317.5" y2="64.77" width="0.254" layer="16"/>
 <wire x1="330.2" y1="57.785" x2="330.2" y2="64.77" width="0.254" layer="16"/>
-<wire x1="302.895" y1="57.785" x2="296.715" y2="63.185" width="0" layer="19" extent="1-1"/>
+<via x="300.99" y="55.88" extent="1-16" drill="0.381"/>
+<wire x1="300.99" y1="55.88" x2="296.545" y2="60.325" width="0.254" layer="16"/>
+<via x="296.545" y="60.325" extent="1-16" drill="0.381"/>
+<wire x1="296.545" y1="60.325" x2="296.545" y2="63.015" width="0.254" layer="1"/>
+<wire x1="296.545" y1="63.015" x2="296.715" y2="63.185" width="0.254" layer="1"/>
+<wire x1="289.56" y1="44.45" x2="289.56" y2="43.18" width="0.4064" layer="1"/>
 </signal>
 <signal name="IN1L+">

Commit message: up
Parts:
- added U$7, U$8: TOGGLE, monome-inc:100SP1T2B4M7RE
- moved C59 86.3 mm to (304.8, 15.9), turned to 0 degrees
- moved R34 81.3 mm to (304.2, 19.7)
- moved R35 81.3 mm to (306.1, 19.7)
- moved C34 1.27 mm to (297.2, 12.7)
- moved U19 1.27 mm to (297.2, 18.4)
Routing:
- net N$43: track 13.4 -> 120.2 mm
- net N$49: track 112.8 -> 9.02 mm
- net +5V: track 670.6 -> 682.6 mm, vias 20 -> 21
- net KEY3^: track 80.8 -> 85.5 mm
- net MODE-KEY^: track 73.2 -> 75.6 mm
- net KEY2^: track 87.3 -> 88.5 mm
- net KEY1^: track 80.4 -> 81.7 mm
- net N$8: track 78.1 -> 76.9 mm
- net N$30: track 20.3 -> 19.0 mm
- net N$23: track 35.4 -> 34.1 mm
- net N$11: track 56.8 -> 55.5 mm
- net KEY0^: track 82.2 -> 83.5 mm
- net N$13: track 26.8 -> 27.5 mm

Commit message: new face
Parts:
- removed U$8: TOGGLE, monome-inc:100SP1T2B4M7RE
- added C140, C141, C156, C157, C159, C160, C196, C197, C207, C208, C210, C211: 10u, rc-master-smd:C1206/T
- added C155, C158, C161, C192, C193, C194, C195, C198, C209: 100n, rc-master-smd:C0603
- added C162, C164, C165: 100u, rc-master-smd:C1206/T
- added C163, C191: 1u, rc-master-smd:C0603
- added IC10, IC11, IC12, IC13, IC14, IC4: AD8607R, analog-devices:SO8
- added J13: PHA2U, monome-inc:PHA2U
- added R117, R119, R120, R121, R122, R123, R124, R126, R127, R128, R156, R157, R158, R159, R160, R161, R166, R176, R177, R178, R179, R180, R181, R183, R184, R185, R68, R69: 100k, rc-master-smd:R0603
- added R118, R125, R175, R182: 50k, rc-master-smd:R0603
- added R129, R130, R132, R154: 3k9, rc-master-smd:R0603
- added R131, R155: 5k, rc-master-smd:R0603
- added R186, R187: 5M, rc-master-smd:R0603
- U$7: value TOGGLE -> (none); device monome-inc:100SP1T2B4M7RE -> monome-inc:SO08
- moved U$7 81.4 mm to (220.3, 27.9), turned to 270 degrees
- moved P5 20.3 mm to (233.7, 78.7)
- moved P6 20.3 mm to (213.4, 78.7)
Connections:
- removed net HP-LP: P3.10
- removed net HP-LP^: P4.10
- removed net HP-RP: P3.12
- removed net HP-RP^: P4.12
- new net GAINL-1: IC14.6, J13._0, R182.2
- new net GAINL-2: C208.+, IC14.7, R181.2, R187.2
- new net GAINR-1: IC13.6, J13.0, R175.2
- new net GAINR-2: C197.+, IC13.7, R166.2, R186.2
- new net IN-VREF: IC12.1, IC12.2, P7.2, P7.3, P8.2, P8.3, R176.1, R177.1, R183.1, R184.1
- new net N$102: C156.-, R118.1
- new net N$103: IC4.6, R117.1, R118.2
- new net N$107: C141.+, IC4.7, R117.2
- new net N$109: IC10.3, R127.2
- new net N$111: IC4.5, R119.2
- new net N$112: P5.1, R68.1
- new net N$113: IC10.2, R122.2, R123.1
- new net N$114: C159.+, IC10.1, R123.2
- new net N$115: C159.-, R125.1
- new net N$120: IC10.6, R124.1, R125.2
- new net N$121: C157.+, IC10.7, R124.2
- new net N$122: IC10.5, R126.2
- new net N$130: P5.4, R122.1
- new net N$140: C160.+, P5.5
- new net N$141: R129.1, R130.2, U$7.2
- new net N$148: C164.+, R129.2, U$7.1
- new net N$149: C163.1, P6.5
- new net N$150: R132.2, R154.1, U$7.6
- new net N$151: C191.1, P6.6
- new net N$152: C192.2, IC12.3, R156.1, R157.2
- new net N$153: IC13.3, R177.2
- new net N$154: C165.-, R132.1, U$7.7
- new net N$155: IC13.2, R160.2, R161.1
- new net N$156: P6.4, R154.2
- new net N$157: P6.1, R130.1
- new net N$158: C207.+, IC13.1, R161.2
- new net N$159: C207.-, R175.1
- new net N$162: IC13.5, R176.2
- new net N$163: C193.2, IC12.5, R158.1, R159.2
- new net N$164: C196.+, P8.6
- new net N$165: P8.1, R160.1
- new net N$166: IC14.3, R184.2
- new net N$167: IC14.2, R179.2, R180.1
- new net N$168: C210.+, IC14.1, R180.2
- new net N$169: C210.-, R182.1
- new net N$172: IC14.5, R183.2
- new net N$173: P7.1, R179.1
- new net N$174: C211.+, P7.6
- new net N$177: J13.1, R166.1
- new net N$180: J13.2, R186.1
- new net N$181: J13._1, R181.1
- new net N$183: J13._2, R187.1
- new net N$89: IC4.3, R120.2
- new net N$90: IC4.2, R68.2, R69.1
- new net N$91: C140.+, P5.6
- new net N$93: C156.+, IC4.1, R69.2
- new net OUT-VREF: IC12.6, IC12.7, P5.2, P5.3, P6.2, P6.3, R119.1, R120.1, R126.1, R127.1, U$7.3, U$7.5
- new net OUT1-LB: C160.-, C163.2, IC11.6, IC11.7
- new net OUT1-RB: C140.-, C191.2, IC11.1, IC11.2
- net +5VA: now also C155.2, C158.2, C161.2, C162.+, C194.2, C195.2, C198.2, C209.2, IC10.8, IC11.8, IC12.8, IC13.8, IC14.8, IC4.8, R156.2, R158.2, U$7.8
- net AGND: now also C155.1, C158.1, C161.1, C162.-, C192.1, C193.1, C194.1, C195.1, C198.1, C209.1, IC10.4, IC11.4, IC12.4, IC13.4, IC14.4, IC4.4, R121.1, R128.1, R131.1, R155.2, R157.1, R159.1, R178.1, R185.1, U$7.4
- net HP-L^: now also C165.+, R155.1
- net HP-R^: now also C164.-, R131.2
- net IN1-LP^: now also C211.-
- net IN1-L^: now also C208.-, R185.2
- net IN1-RP^: now also C196.-
- net IN1-R^: now also C197.-, R178.2
- net OUT1-LP^: now also IC11.5
- net OUT1-L^: now also C157.-, R128.2
- net OUT1-RP^: now also IC11.3
- net OUT1-R^: now also C141.-, R121.2
Routing:
- net +5VA: track 187.1 -> 461.8 mm, vias 8 -> 20
- net OUT-VREF: track 0.00 -> 151.0 mm
- net IN-VREF: track 0.00 -> 111.7 mm
- net GAINR-2: track 0.00 -> 105.0 mm, vias 0 -> 4
- net GAINR-1: track 0.00 -> 98.8 mm, vias 0 -> 4
- net GAINL-2: track 0.00 -> 85.7 mm, vias 0 -> 2
- net GAINL-1: track 0.00 -> 78.4 mm, vias 0 -> 2
- net N$156: track 0.00 -> 75.6 mm
- net IN1-L^: track 0.00 -> 70.8 mm, vias 0 -> 4
- net IN1-R^: track 0.00 -> 68.7 mm, vias 0 -> 6
- net IN1-RP^: track 0.00 -> 68.4 mm, vias 0 -> 6
- net N$157: track 0.00 -> 66.0 mm
- net N$165: track 0.00 -> 65.9 mm
- net AGND: track 213.8 -> 274.7 mm, vias 48 -> 64
- net N$112: track 0.00 -> 57.7 mm
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Other:
- board text added: "130507"
- board text removed: "130128"

Commit message: cad and circuits and text
Parts:
- removed U$7: (no value), monome-inc:SO08
- added IC15: tda1308, monome-inc:SO08
- moved J20 1.80 mm to (316.2, 92.7)
- moved R148 1.80 mm to (351.8, 94.6)
- moved R149 1.80 mm to (351.8, 92.7)
- moved R150 1.80 mm to (363.2, 95.6)
- moved R151 1.80 mm to (363.2, 93.7)
- moved R152 1.80 mm to (363.2, 97.5)
- moved C70 1.80 mm to (280.0, 43.2)
- moved C71 1.80 mm to (280.0, 45.7)
- moved U23 1.80 mm to (311.8, 62.9)
- moved U24 1.80 mm to (324.5, 62.9)
- moved R31 1.80 mm to (264.2, 9.53)
- moved R33 1.80 mm to (284.5, 9.53)
- moved C63 1.80 mm to (299.7, 37.5)
- moved D4 1.80 mm to (308.0, 66.7)
- moved D5 1.80 mm to (320.7, 66.7)
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Connections:
- net +5VA: now also IC15.8; no longer U$7.8
- net AGND: now also IC15.4; no longer U$7.4
- net N$141: now also IC15.2; no longer U$7.2
- net N$148: now also IC15.1; no longer U$7.1
- net N$150: now also IC15.6; no longer U$7.6
- net N$154: now also IC15.7; no longer U$7.7
- net OUT-VREF: now also IC15.3, IC15.5; no longer U$7.3, U$7.5
Other:
- board size 370.8 x 111.8 mm -> 373.4 x 111.1 mm
- board text added: "L bracket 0.0625""
- board text added: "captive spacer 0.125""
- board text added: "mez space 0.5""
- board text added: "mez space 0.75""
- board text added: "outer 0.0375""
- board text added: "plate 0.1875""
