File: circuit/aleph-dev/aleph.brd (EAGLE design)
At the start: 372.1 x 110.5 mm, 571 parts, among them IC1 AD8567, IC10 AD8606, IC11 AD8606, IC12 AD8606, IC13 AD8606, IC14 AD8606, IC15 AD8606, IC16 AD8607R, IC2 AD8606, IC3 AD8606, IC4 AD8606, IC5 AD8606, IC6 AD8606, IC7 AD8606, IC8 AD8606, IC9 AD8606, J1 STEREOSW3GND, J10 PHA2U, J11 USBA-VERT, J12 STX-3680, J13 STX-3680, J14 STX-3680, J15 STX-3680, J16 STX-3680, J17 STX-3680, J18 STX-3680, J19 STX-3680, J2 NSJ12HF, J20 F-2X03-DIL-100, J21 STEREOSW3GND, J22 STEREOSW3GND, J3 NSJ12HF, J4 NSJ12HF, J5 NSJ12HF, J6 SJ1-3533NG, J8 PJ-102AH/BH, J9 PHA2U, K1 PVA1, K2 PVA1, K3 PVA1, K4 PVA1, P1 M-1X05-SIP-100-32, P10 M-2X03-DIL-100, P12 M-1X03-SIP-100-40, P2 EVJ-POT, P3 EVJ-POT, P4 EVJ-POT, P5 EVJ-POT, P6 F-2X06-DIL-100, P7 M-2X06-DIL-100, P8 M-2X14-DIL-100, P9 M-2X14-DIL-100, SW1 PANASONIC-EVQ, U1 BAS70-04, U10 FDS9431A, U11 BAS70-04, U12 BAS70-04, U13 BAS70-04, U14 BAS70-04, U15 AT32UC3A0512, U16 CY62167EV30-Z, U17 AD1939, U2 LMR62014, U21 AD7923, U22 LM4040M3, U23 MT48LC32M16A2tg-75, U24 AD5686R, U25 74HC14D, U26 SN74LVC2G14, U3 BAS70-04, U4 TPS2020, U5 LM2678, U6 ATMEGA32U4-AU, U7 ADP3339, U8 TPA6111A2, U9 ADP3339, X1 16mhz, Y1 ASFL1-27mhz, Y2 12mhz, Y3 ASFL1-12.288mhz

Commit message: notes from sept proto build;
Connections:
- net N$120 renamed U-MOSI
- net N$121 renamed U-SCK
- net N$14 renamed U-MISO
Changed lines of the file:
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@@
 <layer number="14" name="Route14" color="1" fill="6" visible="no" active="no"/>
 <layer number="15" name="Route15" color="4" fill="6" visible="no" active="no"/>
-<layer number="16" name="Bottom" color="1" fill="1" visible="no" active="yes"/>
+<layer number="16" name="Bottom" color="1" fill="1" visible="yes" active="yes"/>
 <layer number="17" name="Pads" color="2" fill="1" visible="yes" active="yes"/>
 <layer number="18" name="Vias" color="2" fill="1" visible="yes" active="yes"/>
@@
 <wire x1="127" y1="75.2475" x2="127" y2="74.295" width="0.2032" layer="16"/>
 </signal>
-<signal name="N$14">
+<signal name="U-MISO">
 <contactref element="P1" pad="2"/>
 <contactref element="U6" pad="11"/>
@@
 <wire x1="110.045" y1="78.55" x2="106.68" y2="81.915" width="0.2032" layer="1"/>
 </signal>
-<signal name="N$120">
+<signal name="U-MOSI">
 <contactref element="P1" pad="3"/>
 <contactref element="U6" pad="10"/>
@@
 <wire x1="109.88" y1="79.35" x2="107.315" y2="81.915" width="0.2032" layer="1"/>
 </signal>
-<signal name="N$121">
+<signal name="U-SCK">
 <contactref element="P1" pad="4"/>
 <contactref element="U6" pad="9"/>
