File: circuit/aleph-dev/aleph.brd (EAGLE design)
At the start: 373.4 x 111.1 mm, 520 parts, among them IC1 AD8606, IC10 AD8607R, IC11 AD8607R, IC12 AD8607R, IC13 AD8607R, IC14 AD8607R, IC15 tda1308, IC2 AD8606, IC3 AD8606, IC4 AD8607R, IC5 AD8606, IC6 AD8606, IC7 AD8607R, IC8 AD8606, IC9 AD8567, J1 SJ1-3533NG, J10 PHA2U, J11 NSJ12HF, J12 NSJ12HF, J13 PHA2U, J15 STX-3680, J16 STX-3680, J17 STX-3680, J18 STX-3680, J19 STX-3680, J2 PJ-102AH/BH, J20 STX-3680, J21 STX-3680, J22 STX-3680, J3 STEREOSW2GND, J4 NSJ12HF, J5 NSJ12HF, J6 STEREOSW2GND, J7 STEREOSW2GND, J8 USBA-VERT, K0 PVA1, K1 PVA1, K2 PVA1, K3 PVA1, P1 M-2X14-DIL-100, P2 M-2X14-DIL-100, P3 M-2X09-DIL-100, P4 M-2X09-DIL-100, P5 EVJ-POT, P6 EVJ-POT, P7 EVJ-POT, P8 EVJ-POT, U1 AT32UC3A0512, U10 LM4040M3, U14 AD1939, U17 AD5686R, U18 FDS9431A, U19 74HC14D, U2 FT232RL, U20 SN74LVC2G14, U21 LM2674, U22 BAS70-04, U23 BAS70-04, U24 BAS70-04, U25 BAS70-04, U3 CY62167EV30-Z, U4 TPS2020, U5 AD7923, U6 LM2678, U7 ADP3339, U8 ADP3339, U9 MT48LC32M16A2tg-75, Y1 12mhz, Y2 ASFL1-27mhz, Y3 ASFL1-12.288mhz

Commit message: circuit updates, cad, txt, etc
Parts:
- removed C175: 15u, rc-master-smd:C6032/T
- removed D8: MBRS130LT3, diode:SMB403A
- removed IC11: AD8607R, analog-devices:SO8
- removed L9: LPS4018-68uh, inductor-coilcraft:LPS4018
- removed LED5, LED6, LED8: (no value), led:CHIPLED_0805
- removed R123, R124, R126, R127, R128, R166, R181: 100k, rc-master-smd:R0603
- removed R125: 50k, rc-master-smd:R0603
- removed R131, R155: 5k, rc-master-smd:R0603
- removed R167, R168: 0, rc-master-smd:R0603
- removed R186, R187: 5M, rc-master-smd:R0603
- removed U2: FT232RL, ftdi-chip:SSOP28
- removed U21: LM2674, monome-inc:SO08
- added C212, C213, C216: 1u, rc-master-smd:C0603
- added C214: 12p, rc-master-smd:C0603
- added C215: 4u7, rc-master-smd:C1206/T
- added C217: 100n, rc-master-smd:C0603
- added C218: 4.7u, rc-master-smd:C1206/T
- added D9: MBR0520L, diode:SOD123
- added H1, H10, H11, H12, H13, H2, H3, H4, H5, H6, H7, H8, H9: MOUNT440, monome-inc:120-PAD-NS
- added J14: F-2X03-DIL-100, con-headers-jp:DIL-100-2X03
- added L11: XAL7030-103, monome-inc:XAL7030-103
- added P10: M-1X05-SIP-100-32, con-headers-jp:SIP-100-05-32
- added P9: M-2X03-DIL-100, con-headers-jp:DIL-100-2X03
- added Q2: J201, monome-inc:SOT95P280X135-3N
- added U$7: TPA6111A2, monome-inc:SO08
- added U$8: ATMEGA32U4-AU, monome-inc:TQFP44
- added U$9: LMR62014, monome-inc:SOT23-5
- added U12, U13: BAS70-04, diode:SOT23
- added X1: 16mhz, monome-inc:NX5032
- C141, C156, C159, C160: value 10u -> 100n; device rc-master-smd:C1206/T -> rc-master-smd:C0603
- C155, C158, C52: value 100n -> 10u; device rc-master-smd:C0603 -> rc-master-smd:C1206/T
- C162: value 100u -> 10u
- C164, C165: value 100u -> 68u
- C176: value 68u -> 2.2u; device rc-master-smd:C7343/T -> rc-master-smd:C1206
- C177: value 10n -> 220p
- C194: value 100n -> 12p
- C54: value 4.7u -> 10u
- IC15: value tda1308 -> AD8607R; device monome-inc:SO08 -> analog-devices:SO8
- P3: value M-2X09-DIL-100 -> F-2X06-DIL-100; device con-headers-jp:DIL-100-2X09 -> con-headers-jp:DIL-100-2X06
- P4: value M-2X09-DIL-100 -> M-2X06-DIL-100; device con-headers-jp:DIL-100-2X09 -> con-headers-jp:DIL-100-2X06
- R117: value 100k -> 6k8
- R118: value 50k -> 3M
- R119: value 100k -> 2k2
- R120: value 100k -> 51k
- R121: value 100k -> 117k
- R122: value 100k -> 13k3
- R129, R130, R132, R154: value 3k9 -> 20k
- R15: value 4.7k -> 22
- R22: value 10k -> 22
- R51, R54, R57, R60: value 10k -> 100k
- moved C159 223.0 mm to (5.40, 76.8)
- moved C161 216.4 mm to (11.4, 81.9)
- moved C162 216.4 mm to (11.4, 84.5)
- moved C164 216.4 mm to (6.35, 84.5)
- moved C165 216.4 mm to (17.8, 84.5)
- moved R129 216.4 mm to (6.35, 79.4)
- moved R130 216.4 mm to (4.45, 79.4)
- moved R132 216.4 mm to (16.5, 78.1)
- moved R154 216.4 mm to (18.4, 78.1)
- moved IC15 214.6 mm to (11.4, 70.2)
- moved C160 211.0 mm to (11.4, 74.0), turned to 0 degrees
- moved R118 128.2 mm to (219.1, 167.0), turned to 0 degrees
- moved R117 127.4 mm to (219.1, 171.4), turned to 0 degrees
- moved R60 120.7 mm to (214.6, 36.5), turned to 90 degrees
- moved C52 117.6 mm to (219.7, 152.4), flipped to the top
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Connections:
- removed net FTDI-CTS: U1.34, U2.3
- removed net FTDI-RTS: U1.32, U2.11
- removed net FTDI-RX: U1.25, U2.1
- removed net FTDI-TX: U1.27, U2.5
- removed net HP-L: J3.R, P3.9
- removed net HP-L^: C165.+, P4.9, R155.1
- removed net HP-R: J3.T, P3.11
- removed net HP-R^: C164.-, P4.11, R131.2
- removed net HPL+: U14.6
- removed net HPL-: U14.7
- removed net HPR+: U14.8
- removed net HPR-: U14.9
- removed net IN1-L: J4.TT, P3.5
- removed net IN1-LP: L3.2, P3.6
- removed net IN1-LP^: C211.-, P4.6
- removed net IN1-L^: C208.-, P4.5, R185.2
- removed net IN1-R: J5.TT, P3.7
- removed net IN1-RP: L4.2, P3.8
- removed net IN1-RP^: C196.-, P4.8
- removed net IN1-R^: C197.-, P4.7, R178.2
- removed net N$177: J13.1, R166.1
- removed net N$180: J13.2, R186.1
- removed net N$181: J13._1, R181.1
- removed net N$183: J13._2, R187.1
- removed net N$33 (its old number): J17.1, R57.1
- removed net OUT1-L: J4.TB, P3.1
- removed net OUT1-LB: C160.-, C163.2, IC11.6, IC11.7
- removed net OUT1-LP: C115.-, P3.2, R97.1
- removed net OUT1-LP^: IC11.5, P4.2
- removed net OUT1-L^: C157.-, P4.1, R128.2
- removed net OUT1-R: J5.TB, P3.3
- removed net OUT1-RB: C140.-, C191.2, IC11.1, IC11.2
- removed net OUT1-RP: C109.-, P3.4, R89.1
- removed net OUT1-RP^: IC11.3, P4.4
- removed net OUT1-R^: C141.-, P4.3, R121.2
- removed net TFS0: DSP1.P$69, R168.2, U14.22
- removed net TSCLK0: DSP1.P$72, R167.2, U14.21
- new net CTS: U$8.12, U1.34
- new net HPL: IC15.5, P3.1
- new net HPL-J: C165.+, J3.R
- new net HPL^: P4.1, P6.4
- new net HPR: IC15.3, P3.3
- new net HPR-J: C164.-, J3.T
- new net HPR^: P4.3, P6.1
- new net IN1L: L3.2, P3.9
- new net IN1L-J: J4.TT, P3.10
- new net IN1L-J^: C211.-, P4.10
- new net IN1L^: C208.-, P4.9, R185.2
- new net IN1R: L4.2, P3.11
- new net IN1R-J: J5.TT, P3.12
- new net IN1R-J^: C196.-, P4.12
- new net IN1R^: C197.-, P4.11, R178.2
- new net N$160: C216.2, U$8.6
- new net N$161: J9.VCC, U$8.7
- new net N$91: IC4.3, P5.4
- new net OUT1L: C115.-, P3.5, R97.1
- new net OUT1L-J: J4.TB, P3.2
- new net OUT1L-J^: C155.-, P4.2, R57.2
- new net OUT1L^: C157.-, C163.2, P4.5
- new net OUT1R: C109.-, P3.7, R89.1
- new net OUT1R-J: J5.TB, P3.4
- new net OUT1R-J^: C158.-, P4.4, R69.2
- new net OUT1R^: C140.-, C191.2, P4.7
- new net RTS: U$8.22, U1.32
- new net RX: U$8.21, U1.25
- new net TX: U$8.20, U1.27
- new net U_RES: P10.5, U$8.13
- net +12V: now also C177.2, C218.+, D9.C, P2.2, R121.2; no longer C176.+, L9.2, P2.24, U21.4
- net +3V3: now also P2.3, U12.2, U13.2; no longer P2.25, U2.4
- net +5V: now also C176.1, C217.2, L11.P$1, P2.4, U$8.14, U$8.2, U$8.24, U$8.34, U$8.42, U$8.44, U$9.4, U$9.5; no longer P2.26, U2.20
- net +5VA: now also C141.2, C156.2, C160.2, P3.6, P4.6, U$7.8; no longer C155.2, C158.2, C194.2, IC11.8, R51.2, R54.2, R57.2, R60.2
- net AGND: now also C141.1, C156.1, C159.1, C160.1, C52.-, J11.RB, J11.RT, J12.RB, J12.RT, J14.1, J14.2, J4.RB, J4.RT, J5.RB, J5.RT, P3.8, P4.8, P9.1, P9.2, R118.2, R119.2, R120.2, R57.1, R69.1, U$7.4, U$7.5; no longer C155.1, C158.1, C194.1, IC11.4, P3.13, P3.14, P4.13, P4.14, R121.1, R128.1, R131.1, R155.2
- net CVOUT1: now also J14.6; no longer P3.15
- net CVOUT1^: now also P9.6; no longer P4.15
- net CVOUT2: now also J14.4; no longer P3.16
- net CVOUT2^: now also P9.4; no longer P4.16
- net CVOUT3: now also J14.5; no longer P3.18
- net CVOUT3^: now also P9.5; no longer P4.18
- net CVOUT4: now also J14.3; no longer P3.17
- net CVOUT4^: now also P9.3; no longer P4.17
- net ENC0A^: now also P2.13; no longer P2.7
- net ENC0B^: now also P2.14; no longer P2.8
- net ENC1A^: now also P2.11; no longer P2.5
- net ENC1B^: now also P2.12; no longer P2.6
- net ENC2A^: now also P2.9; no longer P2.3
- net ENC2B^: now also P2.10; no longer P2.4
- net ENC3A^: now also P2.7; no longer P2.1
- net ENC3B^: now also P2.8; no longer P2.2
- net GAINL-2: no longer R181.2, R187.2
- net GAINR-2: no longer R166.2, R186.2
- net GND: now also C176.2, C194.1, C214.1, C216.1, C217.1, C218.-, P10.1, P2.1, P2.5, P2.6, R122.1, U$8.15, U$8.23, U$8.35, U$8.43, U$8.5, U$9.2, U12.1, U13.1; no longer C175.-, C176.-, C52.1, D8.A, P2.23, P2.27, P2.28, R22.2, U2.18, U2.21, U2.25, U2.7, U21.6
- net KEY0^: now also P2.18; no longer P2.12
- net KEY1^: now also P2.17; no longer P2.11
- net KEY2^: now also P2.16; no longer P2.10
- net KEY3^: now also P2.15; no longer P2.9
- net MODE-KEY^: now also P2.19; no longer P2.13
- net MODE-LED^: now also P2.20; no longer P2.14
- net N$102: now also C158.+, IC10.7, R60.2; no longer C156.-, R118.1
- net N$103: now also IC10.6, R60.1, R68.2; no longer IC4.6, R117.1, R118.2
- net N$107: now also C159.2, U$7.3; no longer C141.+, IC4.7, R117.2
- net N$109: now also C194.2, U$8.16, X1.P$1; no longer IC10.3, R127.2
- net N$111: now also C212.2, IC15.1, IC15.2; no longer IC4.5, R119.2
- net N$112: now also C214.2, U$8.17, X1.P$2; no longer P5.1, R68.1
- net N$113: now also C213.2, IC15.6, IC15.7; no longer IC10.2, R122.2, R123.1
- net N$114: now also C213.1, R154.2; no longer C159.+, IC10.1, R123.2
- net N$115: now also C212.1, R130.1; no longer C159.-, R125.1
- net N$12: now also J9.DP, R22.1; no longer J9.DM, U2.16
- net N$120: now also P10.3, U$8.10; no longer IC10.6, R124.1, R125.2
- net N$121: now also P10.4, U$8.9; no longer C157.+, IC10.7, R124.2
- net N$122: now also Q2.1, R118.1; no longer IC10.5, R126.2
- net N$13: now also R22.2, U$8.4; no longer J9.DP, U2.15
- net N$130: now also Q2.2, R119.1; no longer P5.4, R122.1
- net N$133: now also D9.A, L11.P$2, U$9.1; no longer C177.1, U21.1
- net N$134: now also C177.1, R121.1, R122.2, U$9.3; no longer C177.2, D8.C, L9.1, U21.8
- net N$14: now also P10.2, U$8.11; no longer C52.2, U2.17
- net N$140: now also C215.-, Q2.3, R117.2; no longer C160.+, P5.5
- net N$141: now also U$7.2; no longer IC15.2
- net N$148: now also U$7.1; no longer IC15.1
- net N$150: now also U$7.6; no longer IC15.6
- net N$154: now also U$7.7; no longer IC15.7
- net N$156: now also C215.+, R120.1; no longer P6.4, R154.2
- net N$157: now also C52.+, R117.1; no longer P6.1, R130.1
- net N$17: now also R15.1, U$8.3; no longer J9.VCC, R15.2
- net N$41: now also C157.+, P5.5; no longer J16.1, R54.1
- net N$47: now also IC10.3, P5.1; no longer J15.1, R51.1
- net N$51: now also IC4.1, IC4.2, IC4.5; no longer J18.1, R60.1
- net N$6: now also J9.DM, R15.2; no longer R15.1, R22.1, U2.19
- net N$89: now also C155.+, IC4.7, R51.2; no longer IC4.3, R120.2
- net N$90: now also IC4.6, R51.1, R54.2; no longer IC4.2, R68.2, R69.1
- net N$93: now also IC10.1, IC10.2, IC10.5; no longer C156.+, IC4.1, R69.2
- net OLED-DC^: now also P2.21; no longer P2.15
- net OLED-RES^: now also P2.22; no longer P2.16
- net OUT-VREF: now also R54.1, R68.1; no longer IC15.3, IC15.5, R119.1, R120.1, R126.1, R127.1
- net POWER_ON: no longer U21.5
- net RFS0: now also DSP1.P$69, U14.22; no longer R168.1
- net RSCLK0: now also DSP1.P$72, U14.21; no longer R167.1
- net SCL: now also U13.3
- net SDA: now also U12.3
- net SPI1-CS0^: now also P2.23; no longer P2.17
- net SPI1-CS1^: now also P2.24; no longer P2.18
- net SPI1-MISO^: now also P2.26; no longer P2.20
- net SPI1-MOSI^: now also P2.27; no longer P2.21
- net SPI1-SCK^: now also P2.28; no longer P2.22
- net UNREG_IN: no longer C175.+, U21.7
Routing:
- net OUT-VREF: track 151.0 -> 17.4 mm
- net GAINR-1: track 98.8 -> 0.00 mm, vias 4 -> 0
- net GAINR-2: track 105.0 -> 8.58 mm, vias 4 -> 0
- net +5VA: track 461.8 -> 375.4 mm, vias 20 -> 16
- net IN1-R: track 83.2 -> 0.00 mm
- net OUT1-R: track 77.3 -> 0.00 mm
- net GAINL-2: track 85.7 -> 8.58 mm, vias 2 -> 0
- net N$156: track 75.6 -> 0.00 mm
- net IN1-L^: track 70.8 -> 0.00 mm, vias 4 -> 0
- net GAINL-1: track 78.4 -> 9.27 mm, vias 2 -> 0
- net IN1-R^: track 68.7 -> 0.00 mm, vias 6 -> 0
- net CVOUT1^: track 210.8 -> 142.4 mm
- net IN1-RP^: track 68.4 -> 0.00 mm, vias 6 -> 0
- net N$157: track 66.0 -> 0.00 mm
- net HP-L: track 65.1 -> 0.00 mm
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- added copper zone on layer 1, net N$16
- added copper zone on layer 1, net N$32
Other:
- board size 373.4 x 111.1 mm -> 372.1 x 110.5 mm
- board text added: "130724"
- board text added: "outer 0.05""
- board text added: "plate 0.15" lip 0.0375"
- board text added: "spacer 0.125""
- board text removed: "130315"
- board text removed: "C"
- board text removed: "GND"
- board text removed: "HPL"
- board text removed: "HPR"
- board text removed: "IN1L"
- board text removed: "IN1R"
- board text removed: "J"
- board text removed: "OUT1L"
- board text removed: "OUT1R"
- board text removed: "captive spacer 0.125""
- board text removed: "outer 0.0375""
- board text removed: "plate 0.1875""

Commit message: circuit analog fixes
Parts:
- removed C215: 4u7, rc-master-smd:C1206/T
- removed C52: 10u, rc-master-smd:C1206/T
- removed IC4: AD8607R, analog-devices:SO8
- removed Q2: J201, monome-inc:SOT95P280X135-3N
- removed R117: 6k8, rc-master-smd:R0603
- removed R118: 3M, rc-master-smd:R0603
- removed R119: 2k2, rc-master-smd:R0603
- removed R120: 51k, rc-master-smd:R0603
- added C175: 10u, rc-master-smd:C1206/T
- added H14, H15: MOUNT440, monome-inc:120-PAD-NS
- C156: value 100n -> 10u; device rc-master-smd:C0603 -> rc-master-smd:C1206/T
- R51, R60: value 100k -> 47k
- R54, R68: value 100k -> 10k
- moved C156 6.03 mm to (208.9, 42.5)
Connections:
- removed net N$122: Q2.1, R118.1
- removed net N$130: Q2.2, R119.1
- removed net N$140: C215.-, Q2.3, R117.2
- removed net N$156: C215.+, R120.1
- removed net N$157: C52.+, R117.1
- net +5VA: no longer C156.2, IC4.8
- net AGND: no longer C156.1, C52.-, IC4.4, R118.2, R119.2, R120.2
- net N$102: now also IC10.1; no longer IC10.7
- net N$103: now also IC10.2; no longer IC10.6
- net N$47: now also C156.-; no longer IC10.3
- net N$51: now also C175.+, IC10.5; no longer IC4.1, IC4.2, IC4.5
- net N$89: now also IC10.7; no longer IC4.7
- net N$90: now also IC10.6; no longer IC4.6
- net N$91: now also C175.-; no longer IC4.3
- net N$93: now also C156.+, IC10.3; no longer IC10.1, IC10.2, IC10.5
Routing:
- net N$93: track 7.52 -> 0.00 mm
- net N$51: track 7.52 -> 0.00 mm
- net AGND: track 271.0 -> 267.6 mm, vias 65 -> 63
- net N$90: track 5.39 -> 2.15 mm
- net N$103: track 5.14 -> 2.15 mm
- net +5VA: track 375.4 -> 372.6 mm
- net N$102: track 7.07 -> 5.86 mm
- net N$89: track 7.73 -> 6.52 mm

Commit message: almost final circuit
Parts:
- removed GND0: (no value), pinhead:1X01
- removed IC14, IC15: AD8607R, analog-devices:SO8
- removed JP4: OLED, pinhead:1X20
- removed K0: PVA1, monome-inc:PVA1
- removed L11: XAL7030-103, monome-inc:XAL7030-103
- removed U$7: TPA6111A2, monome-inc:SO08
- removed U$8: ATMEGA32U4-AU, monome-inc:TQFP44
- added C215, C223, C226: 100n, rc-master-smd:C0603
- added C219: 2200p, rc-master-smd:C0603
- added C220, C221: 1n, rc-master-smd:C0603
- added C222: 470n, rc-master-smd:C1206
- added C224: 330p, rc-master-smd:C0603
- added C225, C227: 10u, rc-master-smd:C1206/T
- added C228: 220p, rc-master-smd:C0603
- added C52: 100u, rc-master-smd:C1210/T
- added D10, D11, D12, D8: 1N4148W-7, diode:SOD123
- added D13, D14: MBRS360T3, diode:SMC
- added IC11: AD8607R, analog-devices:SO8
- added IC4: AD8606, analog-devices:SO8
- added JP2: AVR-JTAG, atmel-avr32:AVR-JTAG-10
- added K4: PVA1, monome-inc:PVA1
- added L9: 600, rc-master-smd:L1206
- added LED5, LED6: (no value), led:CHIPLED_0805
- added LED8: (no value), led:CHIPLED_1206
- added R117, R131: 5k76, rc-master-smd:R0603
- added R118: 33, rc-master-smd:R0603
- added R119, R120: 470k, rc-master-smd:R0603
- added R123, R125, R127, R128: 100k, rc-master-smd:R0603
- added R124: 56k, rc-master-smd:R0603
- added R126: 562, rc-master-smd:R0603
- added R155: 82k, rc-master-smd:R0603
- added R166, R193, R195, R196: 10k, rc-master-smd:R0603
- added R167, R168: 39, rc-master-smd:R0603
- added R181, R186: 49k9, rc-master-smd:R0603
- added R187: 47k, rc-master-smd:R0603
- added R188: 330k, rc-master-smd:R0603
- added R189, R190: 22, rc-master-smd:R0603
- added R191: 1k, rc-master-smd:R0603
- added R192: 117k, rc-master-smd:R0603
- added R194: 13k3, rc-master-smd:R0603
- added TP-GND: (no value), pinhead:1X01
- added U11: BAS70-04, diode:SOT23
- added U15: AT32UC3A0512, atmel-avr32:LQFP144
- added U16: CY62167EV30-Z, memory-cypress:TSOP48
- added U21: AD7923, monome-inc:TSSOP16
- added U26: SN74LVC2G14, monome-inc:SOT23-6
- C1, C161: value 100n -> 2.2u; device rc-master-smd:C0603 -> rc-master-smd:C1206
- C10: value 33n -> 4.7u; device rc-master-smd:C0603 -> rc-master-smd:C1206/T
- C100: value 47u -> 10u
- C101, C120, C143, C145, C34, C63, C70, C8, C81, C82, C83, C84: value 100n -> 10u; device rc-master-smd:C0603 -> rc-master-smd:C1206/T
- C102: value 10u -> 390p; device rc-master-smd:C1206/T -> rc-master-smd:C0603
- C103: value 100n -> 5600p
- C104, C110, C122, C95: value 330p -> 100n
- C105: value 680p -> 10u; device rc-master-smd:C0603 -> rc-master-smd:C1206/T
- C106: value 100p -> 120p
- C107: value 220p -> 100n
- C108, C114, C130: value 2200p -> 100n
- C109, C115, C121, C155, C157, C158, C162, C186, C208, C71, C76, C78: value 10u -> 100n; device rc-master-smd:C1206/T -> rc-master-smd:C0603
- C11, C12, C21: value 33n -> 100p
- C111, C123, C98: value 680p -> 100n
- C112, C116, C124: value 100p -> 1u
- C113, C117: value 220p -> 1u
- C118: value 2200p -> 1u
- C119: value 10u -> 1u; device rc-master-smd:C1206/T -> rc-master-smd:C0603
- C125, C126, C142, C193, C195, C50: value 100n -> 10n
- C127, C128, C140, C156, C48, C49: value 10u -> 10n; device rc-master-smd:C1206/T -> rc-master-smd:C0603
- C129: value 220p -> 10n
- C13: value 33n -> 1u
- C132: value 4.7u -> 10n; device rc-master-smd:C1206/T -> rc-master-smd:C0603
- C133: value 100p -> 10n
- C134, C141: value 100n -> 1n
- C135: value 120p -> 100p
- C136, C150: value 120p -> 100n
- C137, C171, C172, C204: value 1n -> 100n
- C138, C152: value 1n -> 10n
- C139, C148, C154, C173: value 100p -> 100n
- C14: value 4.7u -> 10u; device rc-master-smd:C1206 -> rc-master-smd:C1206/T
- C146: value 100n -> 18p
- C147: value 4.7u -> 18p; device rc-master-smd:C1206/T -> rc-master-smd:C0603
- C149: value 100n -> 4.7u; device rc-master-smd:C0603 -> rc-master-smd:C1206/T
- C15: value 33n -> 100n
- C151: value 120p -> 10n
- C153: value 1n -> 4.7u; device rc-master-smd:C0603 -> rc-master-smd:C1206
- C16: value 100n -> 680p
- C163, C191: value 1u -> 33n
- C164: value 68u -> 100n; device rc-master-smd:C1206/T -> rc-master-smd:C0603
- C165: value 68u -> 33n; device rc-master-smd:C1206/T -> rc-master-smd:C0603
- C166, C199: value 4.7u -> 2.7n; device rc-master-smd:C1206/T -> rc-master-smd:C0603
- C167, C200: value 100p -> 33n
- C168, C189: value 100n -> 33n
- C169, C202: value 120p -> 10u; device rc-master-smd:C0603 -> rc-master-smd:C1206/T
- C17: value 4.7u -> 100n; device rc-master-smd:C1206 -> rc-master-smd:C0603
- C170: value 120p -> 1n
- C174, C217, C41, C60, C61, C72: value 100n -> 100p
- C175: value 10u -> 330p; device rc-master-smd:C1206/T -> rc-master-smd:C0603
- C176: value 2.2u -> 2200p; device rc-master-smd:C1206 -> rc-master-smd:C0603
- C177: value 220p -> 2200p
- C178, C209: value 100n -> 330p
- C179: value 10n -> 33n
- C18: value 2.2u -> 120p; device rc-master-smd:C1206 -> rc-master-smd:C0603
- C180: value 10n -> 1n
- C181: value 10n -> 2.2u; device rc-master-smd:C0603 -> rc-master-smd:C1206
- C182: value 10n -> 2.7n
- C183, C67: value 10n -> 100n
- C185: value 100u -> 10n; device rc-master-smd:C1210/T -> rc-master-smd:C0603
- C187: value 5600p -> 100n
- C188: value 390p -> 100n
- C19: value 470p -> 100n
- C190, C210, C211, C3: value 10u -> 4.7u
- C192: value 100n -> 2.7n
- C194: value 12p -> 2.7n
- C196: value 10u -> 470p; device rc-master-smd:C1206/T -> rc-master-smd:C0603
- C197, C207: value 10u -> 33n; device rc-master-smd:C1206/T -> rc-master-smd:C0603
- C2: device rc-master-smd:C1206 -> rc-master-smd:C0603
- C20: value 2.7n -> 120p
- C201, C6: device rc-master-smd:C0603 -> rc-master-smd:C1206
- C203: value 120p -> 4.7u; device rc-master-smd:C0603 -> rc-master-smd:C1206
- C205: value 1n -> 33n
- C206: value 100p -> 2.2u; device rc-master-smd:C0603 -> rc-master-smd:C1206
- C212: value 1u -> 2200p
- C213: value 1u -> 1n
- C214: value 12p -> 1n
- C216, C38, C59: value 1u -> 100p
- C218: value 4.7u -> 22u
- C22: value 2.2u -> 220p; device rc-master-smd:C1206 -> rc-master-smd:C0603
- C23: value 2.7n -> 100n; device rc-master-smd:C0603 -> rc-master-smd:C1206
- C24, C25: value 2.7n -> 10u; device rc-master-smd:C0603 -> rc-master-smd:C1206/T
- C26: value 2.7n -> 100n
- C27: value 33n -> 10n; device rc-master-smd:C0603 -> rc-master-smd:C1206
- C28: value 33n -> 47u; device rc-master-smd:C0603 -> rc-master-smd:C3528/T
- C29, C30: value 33n -> 12p
- C31: value 100n -> 1u
- C32: value 18p -> 100n
- C33: value 18p -> 1u
- C35, C64, C65, C66: value 10n -> 10u; device rc-master-smd:C0603 -> rc-master-smd:C1206/T
- C36: value 1u -> 680p
- C37, C97: value 10n -> 120p
- C39, C62: value 100n -> 120p
- C40: value 2.2u -> 100p; device rc-master-smd:C1206 -> rc-master-smd:C0603
- C42, C85, C86: value 10n -> 220p
- C43: value 22u -> 1u; device rc-master-smd:C1206/T -> rc-master-smd:C0603
- C44: value 470n -> 1u; device rc-master-smd:C1206 -> rc-master-smd:C0603
- C45: value 10n -> 10u; device rc-master-smd:C1206 -> rc-master-smd:C1206/T
- C46: value 47u -> 10u; device rc-master-smd:C3528/T -> rc-master-smd:C1206/T
- C47: value 100n -> 10n; device rc-master-smd:C1206 -> rc-master-smd:C0603
- C5: value 33n -> 10u; device rc-master-smd:C0603 -> rc-master-smd:C1206/T
- C51: value 4.7u -> 100u; device rc-master-smd:C1206/T -> rc-master-smd:C1210/T
- C55: value 1u -> 100n
- C56, C57, C58: value 1u -> 10u; device rc-master-smd:C0603 -> rc-master-smd:C1206/T
- C7, C9: value 100n -> 68u; device rc-master-smd:C0603 -> rc-master-smd:C1206/T
- C73: value 10u -> 100p; device rc-master-smd:C1206/T -> rc-master-smd:C0603
- C74: value 100n -> 10u; device rc-master-smd:C1206 -> rc-master-smd:C1206/T
- C75: value 100u -> 10u; device rc-master-smd:C1210/T -> rc-master-smd:C1206/T
- C77: value 10u -> 120p; device rc-master-smd:C1206/T -> rc-master-smd:C0603
- C79: value 100n -> 47u; device rc-master-smd:C0603 -> rc-master-smd:C1206/T
- C87, C88, C96: value 10n -> 100p
- C93, C94: value 10n -> 680p
- D1: value MBRS360T3 -> MBR0520L; device diode:SMC -> diode:SOD123
- D2: value MBRS360T3 -> zhcs1000; device diode:SMC -> diode:SOT23
- D7: value zhcs1000 -> 1N4148W-7; device diode:SOT23 -> diode:SOD123
- D9: value MBR0520L -> 1N4148W-7
- IC1: value AD8606 -> AD8567; device analog-devices:SO8 -> analog-devices:TSSOP14
- IC10, IC12: value AD8607R -> AD8606
- IC5, IC6, IC8: value AD8606 -> AD8607R
- IC9: value AD8567 -> AD8606; device analog-devices:TSSOP14 -> analog-devices:SO8
- J1: value SJ1-3533NG -> STEREOSW2GND; device monome-inc:SJ1-3533NG -> Audio Jacks 0.25 inch:NEUTRIK-NRJ6HM-1
- J11: value NSJ12HF -> USBA-VERT; device monome-inc:NSJ12HF -> monome-inc:USBA-VERT
- J12: value NSJ12HF -> STX-3680; device monome-inc:NSJ12HF -> monome-inc:STX-3680
- J13: value PHA2U -> STX-3680; device monome-inc:PHA2U -> monome-inc:STX-3680
- J14: value F-2X03-DIL-100 -> STX-3680; device con-headers-jp:DIL-100-2X03 -> monome-inc:STX-3680
- J2: value PJ-102AH/BH -> NSJ12HF; device con-cuistack:PJ-102XH -> monome-inc:NSJ12HF
- J20: value STX-3680 -> F-2X03-DIL-100; device monome-inc:STX-3680 -> con-headers-jp:DIL-100-2X03
- J21, J22: value STX-3680 -> STEREOSW2GND; device monome-inc:STX-3680 -> Audio Jacks 0.25 inch:NEUTRIK-NRJ6HM-1
- J3: value STEREOSW2GND -> NSJ12HF; device Audio Jacks 0.25 inch:NEUTRIK-NRJ6HM-1 -> monome-inc:NSJ12HF
- J6: value STEREOSW2GND -> SJ1-3533NG; device Audio Jacks 0.25 inch:NEUTRIK-NRJ6HM-1 -> monome-inc:SJ1-3533NG
- J7: value STEREOSW2GND -> (none); device Audio Jacks 0.25 inch:NEUTRIK-NRJ6HM-1 -> monome-inc:USB_B
- J8: value USBA-VERT -> PJ-102AH/BH; device monome-inc:USBA-VERT -> con-cuistack:PJ-102XH
- J9: value (none) -> PHA2U; device monome-inc:USB_B -> monome-inc:PHA2U
- JP1: value AVR-JTAG -> OLED; device atmel-avr32:AVR-JTAG-10 -> pinhead:1X20
- L1: value MSS1278 -> XAL7030-103; device inductor-coilcraft:MSS1278 -> monome-inc:XAL7030-103
- L2: value SRR6038-100Y -> 600; device inductor-bourns:SRR6038 -> rc-master-smd:L1206
- L4: value 600 -> MSS1278; device rc-master-smd:L1206 -> inductor-coilcraft:MSS1278
- L8: value 600 -> SRR6038-100Y; device rc-master-smd:L1206 -> inductor-bourns:SRR6038
- LED1, LED2: device led:CHIPLED_1206 -> led:CHIPLED_0805
- LED12: device led:CHIPLED_0805 -> led:CHIPLED_1206
- P1: value M-2X14-DIL-100 -> M-1X05-SIP-100-32; device con-headers-jp:DIL-100-2X14 -> con-headers-jp:SIP-100-05-32
- P10: value M-1X05-SIP-100-32 -> M-2X03-DIL-100; device con-headers-jp:SIP-100-05-32 -> con-headers-jp:DIL-100-2X03
- P2: value M-2X14-DIL-100 -> EVJ-POT; device con-headers-jp:DIL-100-2X14 -> monome-inc:EVJ-POT
- P3: value F-2X06-DIL-100 -> EVJ-POT; device con-headers-jp:DIL-100-2X06 -> monome-inc:EVJ-POT
- P4: value M-2X06-DIL-100 -> EVJ-POT; device con-headers-jp:DIL-100-2X06 -> monome-inc:EVJ-POT
- P6: value EVJ-POT -> F-2X06-DIL-100; device monome-inc:EVJ-POT -> con-headers-jp:DIL-100-2X06
- P7: value EVJ-POT -> M-2X06-DIL-100; device monome-inc:EVJ-POT -> con-headers-jp:DIL-100-2X06
- P8: value EVJ-POT -> M-2X14-DIL-100; device monome-inc:EVJ-POT -> con-headers-jp:DIL-100-2X14
- P9: value M-2X03-DIL-100 -> M-2X14-DIL-100; device con-headers-jp:DIL-100-2X03 -> con-headers-jp:DIL-100-2X14
- R10, R11, R14, R159, R161, R176, R179, R69, R8: value 100k -> 10k
- R100: value 49k9 -> 750k
- R101: value 11k -> 10k
- R102: value 5k49 -> 5k76
- R103: value 3k32 -> 5k76
- R104, R94: value 5k49 -> 10k
- R105: value 604 -> 270
- R106: value 1k65 -> 270
- R107: value 49k9 -> 270
- R108, R109: value 2k74 -> 10k
- R110, R169: value 5k76 -> 10k
- R111: value 5k76 -> 2k74
- R112: value 237 -> 2k74
- R113, R114, R143: value 5k76 -> 4k7
- R115: value 237 -> 1k
- R116: value 750k -> 5k76
- R12, R13, R9: value 100k -> 47k
- R121: value 117k -> 470k
- R122: value 13k3 -> 56k
- R129: value 20k -> 750k
- R130: value 20k -> 5k76
- R132: value 20k -> 100k
- R133, R134, R137, R138: value 5k76 -> 100k
- R135: value 237 -> 82k
- R136, R142: value 5k76 -> 18k
- R139, R141, R173: value 237 -> 100k
- R140: value 5k76 -> 0
- R144: value 237 -> 0
- R145: value 750k -> 4k7
- R146, R73: value 10k -> 100k
- R147, R149, R151, R153: value 10k -> 82k
- R148, R150, R152: value 10k -> 18k
- R15: value 22 -> 120
- R154: value 20k -> 18k
- R156: value 100k -> 82k
- R157: value 100k -> 18k
- R158: value 100k -> 150
- R16, R17, R18: value 0 -> 120
- R160: value 100k -> 22
- R162, R67: value 1k -> 10k
- R163, R171, R172: value 5k76 -> 237
- R164: value 562 -> 237
- R170: value 237 -> 10k
- R174: value 750k -> 49k9
- R175: value 50k -> 49k9
- R177, R180: value 100k -> 0
- R178: value 100k -> 33
- R182: value 50k -> 237
- R183, R184, R185: value 100k -> 237
- R19, R20: value 47k -> 120
- R2: value 82k -> 10k
- R21: value 150 -> 11k
- R22: value 22 -> 5k49
- R23, R47: value 150 -> 5k76
- R24, R25, R26, R49, R50: value 0 -> 5k76
- R27: value 3.32k -> 750k
- R28: value 18k -> 750k
- R29: value 82k -> 3k32
- R3: value 18k -> 10k
- R30: value 82k -> 1k65
- R31: value 18k -> 5k49
- R32, R34: value 82k -> 20k
- R33, R35: value 18k -> 20k
- R36, R54: value 10k -> 2k74
- R37: value 22 -> 150
- R38: value 18k -> 150
- R39: value 82k -> 604
- R4, R5: value 39 -> 10k
- R40: value 18k -> 0
- R41: value 82k -> 0
- R43: value 750k -> 0
- R44, R82: value 11k -> 604
- R45: value 5k49 -> 3.32k
- R46: value 3k32 -> 0
- R48, R75: value 10k -> 5k76
- R51: value 47k -> 5k49
- R52: value 10k -> 3k32
- R53: value 10k -> 1k65
- R55, R72: value 10k -> 0
- R56, R58, R59: value 10k -> 270
- R57: value 100k -> 270
- R6: value 0 -> 10k
- R60: value 47k -> 270
- R61: value 10k -> 150
- R63: value 330k -> 10k
- R64: value 47k -> 10k
- R7: value 0 -> 47k
- R70: value 4k7 -> 11k
- R71: value 4k7 -> 5k49
- R74: value 33 -> 100k
- R76: value 33 -> 5k76
- R77: value 150 -> 470k
- R78: value 10k -> 470k
- R79, R80: value 10k -> 4k7
- R81, R84: value 2k74 -> 5k49
- R83: value 5k49 -> 604
- R85: value 3k32 -> 100k
- R86: value 5k49 -> 100k
- R87: value 604 -> 1k
- R88: value 1k65 -> 1k
- R89: value 49k9 -> 11k
- R90: value 11k -> 3k32
- R91: value 5k49 -> 3k32
- R92: value 5k49 -> 11k
- R93: value 3k32 -> 10k
- R95: value 604 -> 10k
- R96, R99: value 1k65 -> 5k49
- R97: value 49k9 -> 1k65
- R98: value 604 -> 1k65
- U1: value AT32UC3A0512 -> BAS70-04; device atmel-avr32:LQFP144 -> diode:SOT23
- U10: value LM4040M3 -> FDS9431A; device diode:SOT23 -> monome-inc:SO08
- U14: value AD1939 -> BAS70-04; device monome-inc:SQFP-S-10X10-64 -> diode:SOT23
- U17: value AD5686R -> AD1939; device monome-inc:TSSOP16 -> monome-inc:SQFP-S-10X10-64
- U18: value FDS9431A -> TL072D; device monome-inc:SO08 -> linear:SO08
- U19: value 74HC14D -> TL072D; device 74xx-us:SO14 -> linear:SO08
- U20: value SN74LVC2G14 -> TL072D; device monome-inc:SOT23-6 -> linear:SO08
- U22: value BAS70-04 -> LM4040M3
- U23: value BAS70-04 -> MT48LC32M16A2tg-75; device diode:SOT23 -> monome-inc:TSOP54
- U24: value BAS70-04 -> AD5686R; device diode:SOT23 -> monome-inc:TSSOP16
- U25: value BAS70-04 -> 74HC14D; device diode:SOT23 -> 74xx-us:SO14
- U3: value CY62167EV30-Z -> BAS70-04; device memory-cypress:TSOP48 -> diode:SOT23
- U5: value AD7923 -> LM2678; device monome-inc:TSSOP16 -> monome-inc:TO263-7
- U6: value LM2678 -> ATMEGA32U4-AU; device monome-inc:TO263-7 -> monome-inc:TQFP44
- U8: value ADP3339 -> TPA6111A2; device monome-inc:SOT223 -> monome-inc:SO08
- U9: value MT48LC32M16A2tg-75 -> ADP3339; device monome-inc:TSOP54 -> monome-inc:SOT223
- Y1: value 12mhz -> ASFL1-27mhz; device crystal:HC49UP@1 -> crystal:ASFL1
- Y2: value ASFL1-27mhz -> 12mhz; device crystal:ASFL1 -> crystal:HC49UP@1
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- renumbered BM0 to BM2, JP8 to JP3, U$1 to SW1, U$10 to REF-OLED, U$2 to E1, U$3 to E2, U$4 to E4, U$5 to E3, U$6 to S1, U$9 to U2
Connections:
- removed net N$155: IC13.2, R160.2, R161.1
- new net N$122: J3.TB, R19.1
- new net N$130: J3.RB, R18.1
- new net N$140: J2.TB, R15.1
- new net N$156: J2.RB, R17.1
- new net N$157: J3.TT, R20.1
- new net N$170: J2.TT, R16.1
- new net N$171: J10._2, R12.2
- new net N$175: J10._1, R14.2
- new net N$176: J10.2, R9.2
- new net N$177: J10.1, R5.2
- new net N$178: R58.1, U19.7
- new net N$179: R122.2, R123.1, U19.5
- new net N$180: C64.-, IC7.5
- new net N$181: C58.+, IC7.2
- new net N$182: C64.+, P5.1
- new net N$184: D12.C, D9.A, R121.1, U20.1
- new net N$185: D9.C, R107.2
- new net N$186: C84.+, R107.1, R59.1, R95.1, U20.6
- new net N$187: LED11.A, R110.1, U20.2
- new net N$188: LED6.A, R59.2
- new net N$189: LED7.A, R60.2
- new net N$190: R60.1, U20.7
- new net N$191: R124.2, R125.1, U20.5
- new net N$195: D10.A, R119.2, R87.1, R88.1, U18.3
- new net N$196: D10.C, D7.A, R119.1, U18.1
- new net N$197: D7.C, R105.2
- new net N$198: C82.+, R105.1, R56.1, R93.1
- new net N$199: LED9.A, R108.1, U18.2
- new net N$200: LED3.A, R56.2
- net +12V: now also C10.+, C2.1, C228.2, D1.C, IC1.4, P8.24, P9.2, R192.2; no longer C177.2, C178.1, C218.+, D9.C, IC9.4, P1.24, P2.2, R121.2
- net +3V3: now also C111.1, C156.1, C195.1, C68.2, C70.+, C81.+, C89.2, JP1.2, JP2.4, LED12.A, LED8.A, P8.25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; no longer C125.2, C127.+, C35.1, C37.1, C41.1, C70.2, C71.+, JP1.4, JP4.2, LED1.A, LED2.A, P1.25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
- net +3V3A: now also C102.1, C107.2, C14.+, C150.1, C160.1, C162.1, C17.2, C171.2, C19.2, C215.2, C67.2, C78.2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; no longer C103.2, C134.2, C143.1, C145.1, C146.1, C149.2, C168.2, C174.2, C188.1, C190.+, C201.2, C39.2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
- net +3V3C: now also C125.2, C126.2, C127.2, C128.2, C129.2, C132.2, C133.2, C148.1, C158.1, C193.1, L2.2, R143.1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; no longer C179.2, C180.2, C181.2, C182.2, C183.2, C184.2, C189.1, C42.2, C96.1, C97.1, L7.2, R42.1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
- net +5V: now also C1.1, C114.2, C115.2, C120.+, C121.2, C122.2, C130.1, C131.+, C223.2, C225.+, C226.2, C227.+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; no longer C120.1, C121.+, C126.2, C128.+, C176.1, C2.2, C217.2, C3.+, C34.2, C46.+, C47.2, C48.+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
- net +5VA: now also C104.2, C105.+, C110.2, C15.2, C32.2, C53.2, C55.2, C76.2, C8.+, C90.2, C91.2, C92.2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; no longer C141.2, C160.2, C161.2, C162.+, C195.2, C198.2, C209.2, C68.2, C69.+, IC10.8, IC12.8, IC14.8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
- net A-A1: now also U15.118, U16.25; no longer U1.118, U3.25
- net A-A10: now also U15.97, U16.7; no longer U1.97, U3.7
- net A-A11: now also U15.95, U16.6; no longer U1.95, U3.6
- net A-A12: now also U15.91, U16.5; no longer U1.91, U3.5
- net A-A13: now also U15.89, U16.4; no longer U1.89, U3.4
- net A-A14: now also U15.87, U16.3; no longer U1.87, U3.3
- net A-A15: now also U15.67, U16.2; no longer U1.67, U3.2
- net A-A16: now also U15.65, U16.1; no longer U1.65, U3.1
- net A-A17: now also U15.63, U16.48; no longer U1.63, U3.48
- net A-A18: now also U15.61, U16.17; no longer U1.61, U3.17
- net A-A19: now also U15.59, U16.16; no longer U1.59, U3.16
- net A-A2: now also U15.114, U16.24; no longer U1.114, U3.24
- net A-A3: now also U15.112, U16.23; no longer U1.112, U3.23
- net A-A4: now also U15.110, U16.22; no longer U1.110, U3.22
- net A-A5: now also U15.107, U16.21; no longer U1.107, U3.21
- net A-A6: now also U15.105, U16.20; no longer U1.105, U3.20
- net A-A7: now also U15.103, U16.19; no longer U1.103, U3.19
- net A-A8: now also U15.101, U16.18; no longer U1.101, U3.18
- net A-A9: now also U15.99, U16.8; no longer U1.99, U3.8
- net A-D0: now also U15.38, U16.29; no longer U1.38, U3.29
- net A-D1: now also U15.35, U16.31; no longer U1.35, U3.31
- net A-D10: now also U15.1, U16.34; no longer U1.1, U3.34
- net A-D11: now also U15.144, U16.36; no longer U1.144, U3.36
- net A-D12: now also U15.142, U16.39; no longer U1.142, U3.39
- net A-D13: now also U15.140, U16.41; no longer U1.140, U3.41
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Routing:
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Other:
- board text added: "130808"
- board text removed: "130724"

Commit message: spreadsheets and eagle
Parts:
- added P12: M-1X03-SIP-100-40, con-headers-jp:SIP-100-03-40
- C27: device rc-master-smd:C1206 -> rc-master-smd:C0603
- C28: device rc-master-smd:C3528/T -> rc-master-smd:C1206/T
- C29, C30: value 12p -> 8p
- IC11, IC13, IC5, IC6, IC7, IC8: value AD8607R -> AD8606
- L10, L2, L3, L5, L6, L7, L9: device rc-master-smd:L1206 -> rc-master-smd:L0603
- moved H14 1.91 mm to (295.9, 3.17)
- moved C27 1.91 mm to (144.1, 77.5)
Connections:
- new net N$155: DSP1.P$81, P12.3
- new net N$183: DSP1.P$82, P12.2
- net GND: now also P12.1
Routing:
- net N$155: track 0.00 -> 44.9 mm
- net N$183: track 0.00 -> 44.8 mm
- net OUT1R: track 11.1 -> 14.2 mm, vias 0 -> 1
- net RSCLK0: track 26.2 -> 24.4 mm, vias 2 -> 0
- net N$9: track 4.45 -> 2.75 mm
- net DT1SEC: track 35.8 -> 35.3 mm
- net N$7: track 32.0 -> 32.5 mm
- net N$98: track 8.86 -> 9.37 mm
- net N$106: track 8.86 -> 9.37 mm
- net +3V3A: track 46.8 -> 47.3 mm
- net N$144: track 8.86 -> 9.37 mm
- net N$126: track 8.86 -> 9.37 mm
- net +3V3C: track 134.3 -> 134.8 mm
- net AGND: track 311.5 -> 312.0 mm

Commit message: final circuit
Parts:
- R187: value 47k -> 18k
- R188: value 330k -> 47k
- R192: value 117k -> 118k
- R45: value 3.32k -> 3k32
Routing:
- net IN-VREF: track 136.0 -> 131.7 mm, vias 4 -> 3
- net N$33: track 9.51 -> 8.76 mm
- net N$151: track 9.53 -> 8.78 mm
- net GAINR-2: vias 4 -> 2

Commit message: circuits and mechanicals
Parts:
- removed LED9: (no value), led:CHIPLED_0805
- removed R108: 10k, rc-master-smd:R0603
- added C229: 100u, rc-master-smd:C7343-43
- C218: device rc-master-smd:C1206/T -> rc-master-smd:C6032-28/T
- C222: value 470n -> 100n
- C28: value 47u -> 100u; device rc-master-smd:C1206/T -> rc-master-smd:C7343-43
- J1, J21, J22: value STEREOSW2GND -> STEREOSW3GND; device Audio Jacks 0.25 inch:NEUTRIK-NRJ6HM-1 -> monome-inc:NEUTRIK-NRJ6HF-1
- J8: device con-cuistack:PJ-102XH -> monome-inc:PJ-102XH
- LED12, LED8: device led:CHIPLED_1206 -> led:CHIPLED_0805
- R119, R120, R121: value 470k -> 47k
- moved P10 106.4 mm to (355.0, 87.0)
- moved J20 7.62 mm to (62.9, 24.8)
- moved C218 6.87 mm to (146.1, 81.9)
- moved C90 3.81 mm to (233.0, 41.9)
- moved P12 3.81 mm to (61.0, 6.35)
- moved R195 1.93 mm to (115.3, 104.8), turned to 90 degrees
- moved R196 1.91 mm to (116.8, 104.8), turned to 90 degrees
- moved C28 1.42 mm to (151.1, 74.9), flipped to the bottom, turned to 180 degrees
- moved D10 1.27 mm to (226.1, 38.1)
- moved R119 1.27 mm to (226.1, 36.2)
- moved C222 0.64 mm to (142.2, 78.7)
- moved C9 0.64 mm to (17.1, 84.5), turned to 0 degrees
- moved C27 0.32 mm to (143.8, 77.5)
Connections:
- removed net N$199: LED9.A, R108.1, U18.2
- new net A-INT: DSP1.P$32, U15.5
- new net B-INT: DSP1.P$29, U15.3
- net +12V: now also P8.2; no longer P8.24
- net +3V3: now also P8.3; no longer P8.25
- net +5V: now also C229.+, P8.4; no longer P8.26
- net +5VA: no longer R108.2
- net AGND: now also J1.SN, U18.3; no longer J1.S, LED9.C
- net ENC0A: now also P8.13; no longer P8.7
- net ENC0B: now also P8.14; no longer P8.8
- net ENC1A: now also P8.11; no longer P8.5
- net ENC1B: now also P8.12; no longer P8.6
- net ENC2A: now also P8.9; no longer P8.3
- net ENC2B: now also P8.10; no longer P8.4
- net ENC3A: now also P8.7; no longer P8.1
- net ENC3B: now also P8.8; no longer P8.2
- net GND: now also C229.-, J21.SN, J22.SN, P8.1, P8.5, P8.6; no longer J21.S, J22.S, P8.23, P8.27, P8.28
- net HPL-J: now also C9.-; no longer C9.+
- net KEY0: now also P8.18; no longer P8.12
- net KEY1: now also P8.17; no longer P8.11
- net KEY2: now also P8.16; no longer P8.10
- net KEY3: now also P8.15; no longer P8.9
- net MODE-KEY: now also P8.19; no longer P8.13
- net MODE-LED: now also P8.20; no longer P8.14
- net N$154: now also C9.+; no longer C9.-
- net N$195: now also U18.2; no longer U18.3
- net OLED-DC: now also P8.21; no longer P8.15
- net OLED-RES: now also P8.22; no longer P8.16
- net SPI1-CS0: now also P8.23; no longer P8.17
- net SPI1-CS1: now also P8.24; no longer P8.18
- net SPI1-MISO: now also P8.26; no longer P8.20
- net SPI1-MOSI: now also P8.27; no longer P8.21
- net SPI1-SCK: now also P8.28; no longer P8.22
Routing:
- net CVOUT4^: track 152.7 -> 16.8 mm, vias 2 -> 0
- net CVOUT2^: track 141.4 -> 8.47 mm
- net CVOUT1^: track 142.4 -> 10.3 mm
- net CVOUT3^: track 144.7 -> 13.7 mm
- net A-INT: track 0.00 -> 82.2 mm, vias 0 -> 4
- net B-INT: track 0.00 -> 78.0 mm, vias 0 -> 4
- net +12V: track 143.1 -> 113.6 mm
- net CVOUT3: track 19.3 -> 10.3 mm
- net SDA: track 101.9 -> 93.1 mm, vias 3 -> 2
- net +5V: track 684.6 -> 693.1 mm, vias 22 -> 23
- net SPI1-MOSI: track 110.9 -> 118.7 mm
- net SPI1-MISO: track 96.5 -> 103.9 mm
- net SPI1-SCK: track 107.8 -> 115.3 mm
- net N$199: track 6.89 -> 0.00 mm
- net CVOUT2: track 15.3 -> 8.45 mm
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Other:
- outline, holes or cut-outs redrawn
- board text added: "130828"
- board text removed: "130507"
- board text removed: "130808"

Commit message: final circuit build notes
Parts:
- removed LED10, LED11: (no value), led:CHIPLED_0805
- removed R109, R110: 10k, rc-master-smd:R0603
- removed U18, U19, U20: TL072D, linear:SO08
- added IC14, IC15: AD8606, analog-devices:SO8
- added IC16: AD8607R, analog-devices:SO8
Connections:
- removed net N$168: LED10.A, R109.1, U19.2
- removed net N$174: LED5.A, R58.2
- removed net N$181: C58.+, IC7.2
- removed net N$187: LED11.A, R110.1, U20.2
- removed net N$189: LED7.A, R60.2
- net +5VA: now also IC14.8, IC15.8, IC16.4, LED7.A; no longer R109.2, R110.2, U18.8, U19.8, U20.8
- net AGND: now also IC14.3, IC14.4, IC15.3, IC15.4, IC16.3, IC16.5, IC16.6, IC16.8; no longer LED10.C, LED11.C, LED5.C, LED7.C, U18.3, U18.4, U18.5, U18.6, U19.4, U20.4
- net IN1L^: now also IC15.2; no longer U19.3
- net IN1R^: now also IC14.2; no longer U20.3
- net N$153: now also C57.+
- net N$158: now also IC6.2
- net N$162: now also IC15.1; no longer U19.1
- net N$164: now also LED7.C, R60.2; no longer C57.+, IC6.2
- net N$167: now also IC15.6; no longer U19.6
- net N$169: now also C58.+
- net N$172: now also IC7.2
- net N$178: now also IC15.7; no longer U19.7
- net N$179: now also IC15.5; no longer U19.5
- net N$184: now also IC14.1; no longer U20.1
- net N$186: now also IC14.6; no longer U20.6
- net N$190: now also IC14.7; no longer U20.7
- net N$191: now also IC14.5; no longer U20.5
- net N$195: now also IC16.2; no longer U18.2
- net N$196: now also IC16.1; no longer U18.1
Routing:
- net AGND: track 313.3 -> 299.0 mm, vias 84 -> 78
- net +5VA: track 508.9 -> 496.5 mm
- net N$187: track 6.89 -> 0.00 mm
- net N$168: track 6.89 -> 0.00 mm
- net N$181: track 3.64 -> 0.00 mm
- net N$164: track 3.64 -> 0.00 mm
- net N$169: track 2.53 -> 0.18 mm
- net N$195: track 25.1 -> 23.3 mm
- net N$167: track 40.3 -> 38.4 mm
- net IN1L^: track 85.3 -> 83.4 mm
- net N$190: track 31.9 -> 30.1 mm
- net N$186: track 44.4 -> 42.5 mm
- net IN1R^: track 111.0 -> 109.2 mm
- net N$174: track 1.71 -> 0.00 mm
- net N$189: track 1.71 -> 0.00 mm
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