File: circuit/aleph-dev/aleph.brd (EAGLE design)
At the start: 372.1 x 110.5 mm, 571 parts, among them IC1 AD8567, IC10 AD8606, IC11 AD8606, IC12 AD8606, IC13 AD8606, IC14 AD8606, IC15 AD8606, IC16 AD8607R, IC2 AD8606, IC3 AD8606, IC4 AD8606, IC5 AD8606, IC6 AD8606, IC7 AD8606, IC8 AD8606, IC9 AD8606, J1 STEREOSW3GND, J10 PHA2U, J11 USBA-VERT, J12 STX-3680, J13 STX-3680, J14 STX-3680, J15 STX-3680, J16 STX-3680, J17 STX-3680, J18 STX-3680, J19 STX-3680, J2 NSJ12HF, J20 F-2X03-DIL-100, J21 STEREOSW3GND, J22 STEREOSW3GND, J3 NSJ12HF, J4 NSJ12HF, J5 NSJ12HF, J6 SJ1-3533NG, J8 PJ-102AH/BH, J9 PHA2U, K1 PVA1, K2 PVA1, K3 PVA1, K4 PVA1, P1 M-1X05-SIP-100-32, P10 M-2X03-DIL-100, P12 M-1X03-SIP-100-40, P2 EVJ-POT, P3 EVJ-POT, P4 EVJ-POT, P5 EVJ-POT, P6 F-2X06-DIL-100, P7 M-2X06-DIL-100, P8 M-2X14-DIL-100, P9 M-2X14-DIL-100, SW1 PANASONIC-EVQ, U1 BAS70-04, U10 FDS9431A, U11 BAS70-04, U12 BAS70-04, U13 BAS70-04, U14 BAS70-04, U15 AT32UC3A0512, U16 CY62167EV30-Z, U17 AD1939, U2 LMR62014, U21 AD7923, U22 LM4040M3, U23 MT48LC32M16A2tg-75, U24 AD5686R, U25 74HC14D, U26 SN74LVC2G14, U3 BAS70-04, U4 TPS2020, U5 LM2678, U6 ATMEGA32U4-AU, U7 ADP3339, U8 TPA6111A2, U9 ADP3339, X1 16mhz, Y1 ASFL1-27mhz, Y2 12mhz, Y3 ASFL1-12.288mhz

Commit message: blind dsyn code
Parts:
- C146, C147: value 18p -> 22p
- R1, R10, R11, R2: value 10k -> 20k
Changed lines of the file:
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@@
 <layers>
 <layer number="1" name="Top" color="4" fill="1" visible="yes" active="yes"/>
-<layer number="2" name="power" color="1" fill="3" visible="no" active="yes"/>
+<layer number="2" name="power" color="1" fill="3" visible="yes" active="yes"/>
 <layer number="3" name="gnd" color="4" fill="3" visible="no" active="yes"/>
 <layer number="4" name="Route4" color="1" fill="4" visible="no" active="no"/>
@@
 <layer number="17" name="Pads" color="2" fill="1" visible="yes" active="yes"/>
 <layer number="18" name="Vias" color="2" fill="1" visible="yes" active="yes"/>
-<layer number="19" name="Unrouted" color="6" fill="1" visible="no" active="yes"/>
+<layer number="19" name="Unrouted" color="6" fill="1" visible="yes" active="yes"/>
 <layer number="20" name="Dimension" color="13" fill="1" visible="yes" active="yes"/>
 <layer number="21" name="tPlace" color="7" fill="1" visible="yes" active="yes"/>
@@
 <attribute name="VALUE" x="151.13" y="10.16" size="1.016" layer="28" font="vector" ratio="12" rot="MR0"/>
 </element>
-<element name="C146" library="rc-master-smd" package="C0603" value="18p" x="135.89" y="37.465" smashed="yes" rot="MR0">
+<element name="C146" library="rc-master-smd" package="C0603" value="22p" x="135.89" y="37.465" smashed="yes" rot="MR0">
 <attribute name="NAME" x="137.795" y="34.925" size="1.016" layer="26" font="vector" ratio="18" rot="MR0"/>
 <attribute name="VALUE" x="137.16" y="34.925" size="1.016" layer="28" font="vector" ratio="12" rot="MR0"/>
 </element>
-<element name="C147" library="rc-master-smd" package="C0603" value="18p" x="132.08" y="37.465" smashed="yes" rot="MR180">
+<element name="C147" library="rc-master-smd" package="C0603" value="22p" x="132.08" y="37.465" smashed="yes" rot="MR180">
 <attribute name="NAME" x="133.35" y="34.925" size="1.016" layer="26" font="vector" ratio="18" rot="MR0"/>
 <attribute name="VALUE" x="133.35" y="34.925" size="1.016" layer="28" font="vector" ratio="12" rot="MR0"/>
@@
 <element name="C2" library="rc-master-smd" package="C0603" value="100n" x="350.52" y="95.885" smashed="yes" rot="R180">
 <attribute name="NAME" x="347.98" y="96.2025" size="1.016" layer="25" font="vector" ratio="18" rot="R180"/>
-<attribute name="VALUE" x="351.79" y="97.6313" size="0.8128" layer="27" ratio="10" rot="R180"/>
+<attribute name="VALUE" x="346.71" y="96.3613" size="0.8128" layer="27" ratio="10" rot="R180"/>
 </element>
 <element name="R3" library="rc-master-smd" package="R0603" value="10k" x="351.155" y="97.79" smashed="yes">
 <attribute name="NAME" x="349.25" y="98.1075" size="1.016" layer="25" font="vector" ratio="18" rot="R180"/>
-<attribute name="VALUE" x="349.885" y="96.0437" size="0.8128" layer="27" ratio="10"/>
-</element>
-<element name="R1" library="rc-master-smd" package="R0603" value="10k" x="351.155" y="99.695" smashed="yes" rot="R180">
+<attribute name="VALUE" x="346.075" y="97.3137" size="0.8128" layer="27" ratio="10"/>
+</element>
+<element name="R1" library="rc-master-smd" package="R0603" value="20k" x="351.155" y="99.695" smashed="yes" rot="R180">
 <attribute name="NAME" x="349.25" y="100.0125" size="1.016" layer="25" font="vector" ratio="18" rot="R180"/>
-<attribute name="VALUE" x="352.425" y="101.4413" size="0.8128" layer="27" ratio="10" rot="R180"/>
+<attribute name="VALUE" x="348.615" y="100.1713" size="0.8128" layer="27" ratio="10" rot="R180"/>
 </element>
 <element name="R8" library="rc-master-smd" package="R0603" value="10k" x="351.155" y="93.98" smashed="yes">
 <attribute name="NAME" x="349.25" y="94.2975" size="1.016" layer="25" font="vector" ratio="18" rot="R180"/>
-<attribute name="VALUE" x="349.885" y="92.2337" size="0.8128" layer="27" ratio="10"/>
-</element>
-<element name="R11" library="rc-master-smd" package="R0603" value="10k" x="351.155" y="92.075" smashed="yes" rot="R180">
+<attribute name="VALUE" x="346.075" y="93.5037" size="0.8128" layer="27" ratio="10"/>
+</element>
+<element name="R11" library="rc-master-smd" package="R0603" value="20k" x="351.155" y="92.075" smashed="yes" rot="R180">
 <attribute name="NAME" x="349.25" y="92.3925" size="1.016" layer="25" font="vector" ratio="18" rot="R180"/>
-<attribute name="VALUE" x="352.425" y="93.8213" size="0.8128" layer="27" ratio="10" rot="R180"/>
+<attribute name="VALUE" x="348.615" y="92.5513" size="0.8128" layer="27" ratio="10" rot="R180"/>
 </element>
 <element name="R6" library="rc-master-smd" package="R0603" value="10k" x="362.585" y="94.9325" smashed="yes" rot="R180">
 <attribute name="NAME" x="364.49" y="94.2975" size="1.016" layer="25" font="vector" ratio="18"/>
-<attribute name="VALUE" x="363.855" y="96.6788" size="0.8128" layer="27" ratio="10" rot="R180"/>
-</element>
-<element name="R10" library="rc-master-smd" package="R0603" value="10k" x="362.585" y="93.0275" smashed="yes">
+<attribute name="VALUE" x="367.665" y="95.4088" size="0.8128" layer="27" ratio="10" rot="R180"/>
+</element>
+<element name="R10" library="rc-master-smd" package="R0603" value="20k" x="362.585" y="93.0275" smashed="yes">
 <attribute name="NAME" x="364.49" y="92.3925" size="1.016" layer="25" font="vector" ratio="18"/>
-<attribute name="VALUE" x="361.315" y="91.2812" size="0.8128" layer="27" ratio="10"/>
+<attribute name="VALUE" x="365.125" y="92.5512" size="0.8128" layer="27" ratio="10"/>
 </element>
 <element name="R4" library="rc-master-smd" package="R0603" value="10k" x="362.585" y="96.8375" smashed="yes" rot="R180">
 <attribute name="NAME" x="364.49" y="96.2025" size="1.016" layer="25" font="vector" ratio="18"/>
-<attribute name="VALUE" x="363.855" y="98.5838" size="0.8128" layer="27" ratio="10" rot="R180"/>
-</element>
-<element name="R2" library="rc-master-smd" package="R0603" value="10k" x="362.585" y="98.7425" smashed="yes">
+<attribute name="VALUE" x="367.665" y="97.3138" size="0.8128" layer="27" ratio="10" rot="R180"/>
+</element>
+<element name="R2" library="rc-master-smd" package="R0603" value="20k" x="362.585" y="98.7425" smashed="yes">
 <attribute name="NAME" x="364.49" y="98.1075" size="1.016" layer="25" font="vector" ratio="18"/>
-<attribute name="VALUE" x="361.315" y="96.9962" size="0.8128" layer="27" ratio="10"/>
+<attribute name="VALUE" x="365.125" y="98.2662" size="0.8128" layer="27" ratio="10"/>
 </element>
 <element name="L5" library="rc-master-smd" package="L0603" value="600" x="365.125" y="79.375" smashed="yes" rot="R270">
