File: circuit/aleph-dev/out-gain.brd (EAGLE design)
At the start: 33 parts, among them IC10 AD8607R, IC12 AD8607R, IC4 AD8607R, P5 EVJ-POT

Commit message: circuit updates, cad, txt, etc
Parts:
- removed C140, C141, C156, C157, C159, C160: 10u, rc-master-smd:C1206/T
- removed C155, C158, C192, C193, C195: 100n, rc-master-smd:C0603
- removed IC10, IC12, IC4: AD8607R, analog-devices:SO8
- removed P5: EVJ-POT, monome-inc:EVJ-POT
- removed R117, R119, R120, R121, R122, R123, R124, R126, R127, R128, R156, R157, R158, R159, R68, R69: 100k, rc-master-smd:R0603
- removed R118, R125: 50k, rc-master-smd:R0603
- added C1, C2, C5, C7: 10u, rc-master-smd:C1206/T
- added C3, C6: 100n, rc-master-smd:C0603
- added IC2, IC3: AD8607R, analog-devices:SO8
- added P1: EVJ-POT, monome-inc:EVJ-POT
- added R1, R10, R2, R3, R8, R9: 100k, rc-master-smd:R0603
Connections:
- removed net HP-VREF: IC12.6, IC12.7
- removed net N$102: C156.-, R118.1
- removed net N$103: IC4.6, R117.1, R118.2
- removed net N$107: C141.+, IC4.7, R117.2
- removed net N$109: IC10.3, R127.2
- removed net N$111: IC4.5, R119.2
- removed net N$112: P5.1, R68.1
- removed net N$113: IC10.2, R122.2, R123.1
- removed net N$114: C159.+, IC10.1, R123.2
- removed net N$115: C159.-, R125.1
- removed net N$120: IC10.6, R124.1, R125.2
- removed net N$121: C157.+, IC10.7, R124.2
- removed net N$122: IC10.5, R126.2
- removed net N$130: P5.4, R122.1
- removed net N$140: C160.+, P5.5
- removed net N$152: C192.2, IC12.3, R156.1, R157.2
- removed net N$163: C193.2, IC12.5, R158.1, R159.2
- removed net N$89: IC4.3, R120.2
- removed net N$90: IC4.2, R68.2, R69.1
- removed net N$91: C140.+, P5.6
- removed net N$93: C156.+, IC4.1, R69.2
- new net N$1: IC3.3, P1.1
- new net N$10: IC2.3, P1.4
- new net N$11: C7.+, P1.5
- new net N$2: IC3.1, IC3.2, IC3.5
- new net N$3: C2.+, IC3.7, R1.2
- new net N$33: IC2.1, IC2.2, IC2.5
- new net N$4: IC3.6, R1.1, R2.2
- new net N$41: C5.+, IC2.7, R8.2
- new net N$47: IC2.6, R8.1, R9.2
- new net N$8: C1.+, P1.6
- net +5VA: now also C3.2, C6.2, IC2.8, IC3.8; no longer C155.2, C158.2, C195.2, IC10.8, IC12.8, IC4.8, R156.2, R158.2
- net AGND: now also C3.1, C6.1, IC2.4, IC3.4, R10.1, R3.1; no longer C155.1, C158.1, C192.1, C193.1, C195.1, IC10.4, IC12.4, IC4.4, R121.1, R128.1, R157.1, R159.1
- net OUT-VREF: now also P1.2, P1.3, R2.1, R9.1; no longer IC12.1, IC12.2, P5.2, P5.3, R119.1, R120.1, R126.1, R127.1
- net OUT1-LB: now also C7.-; no longer C160.-
- net OUT1-L^: now also C5.-, R10.2; no longer C157.-, R128.2
- net OUT1-RB: now also C1.-; no longer C140.-
- net OUT1-R^: now also C2.-, R3.2; no longer C141.-, R121.2
Routing:
- net OUT-VREF: track 100.4 -> 2.92 mm
- net N$112: track 58.5 -> 0.00 mm
- net N$130: track 40.0 -> 0.00 mm, vias 2 -> 0
- net HP-VREF: track 38.6 -> 0.00 mm
- net AGND: track 29.1 -> 9.54 mm
- net +5VA: track 19.1 -> 2.76 mm
- net N$121: track 11.1 -> 0.00 mm
- net N$107: track 11.1 -> 0.00 mm
- net N$120: track 9.56 -> 0.00 mm
- net N$103: track 9.56 -> 0.00 mm
- net N$140: track 7.86 -> 0.00 mm
- net N$41: track 0.00 -> 7.73 mm
- net N$33: track 0.00 -> 7.52 mm
- net N$2: track 0.00 -> 7.52 mm
- net N$163: track 7.30 -> 0.00 mm
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