File: circuit/aleph-dev/out-gain.sch (EAGLE design)
At the start: 33 parts, among them IC10 AD8607R, IC12 AD8607R, IC4 AD8607R, P5 EVJ-POT

Commit message: circuit updates, cad, txt, etc
Parts:
- removed C140, C141, C156, C157, C159, C160: 10u, rc-master-smd:CP_1206/T
- removed C155, C158, C192, C193, C195: 100n, rc-master-smd:C_0603
- removed IC10, IC12, IC4: AD8607R, analog-devices:AD8607R
- removed P5: EVJ-POT, monome-inc:EVJ-POT
- removed R117, R119, R120, R121, R122, R123, R124, R126, R127, R128, R156, R157, R158, R159, R68, R69: 100k, rc-master-smd:R_0603
- removed R118, R125: 50k, rc-master-smd:R_0603
- added C1, C2, C5, C7: 10u, rc-master-smd:CP_1206/T
- added C3, C6: 100n, rc-master-smd:C_0603
- added IC2, IC3: AD8607R, analog-devices:AD8607R
- added P1: EVJ-POT, monome-inc:EVJ-POT
- added R1, R10, R2, R3, R8, R9: 100k, rc-master-smd:R_0603
Connections:
- removed net HP-VREF: IC12B.IN-, IC12B.OUT
- removed net N$102: C156.-, R118.1
- removed net N$103: IC4B.IN-, R117.1, R118.2
- removed net N$107: C141.+, IC4B.OUT, R117.2
- removed net N$109: IC10A.IN+, R127.2
- removed net N$111: IC4B.IN+, R119.2
- removed net N$112: P5.1, R68.1
- removed net N$113: IC10A.IN-, R122.2, R123.1
- removed net N$114: C159.+, IC10A.OUT, R123.2
- removed net N$115: C159.-, R125.1
- removed net N$120: IC10B.IN-, R124.1, R125.2
- removed net N$121: C157.+, IC10B.OUT, R124.2
- removed net N$122: IC10B.IN+, R126.2
- removed net N$130: P5.4, R122.1
- removed net N$140: C160.+, P5.5
- removed net N$152: C192.2, IC12A.IN+, R156.1, R157.2
- removed net N$163: C193.2, IC12B.IN+, R158.1, R159.2
- removed net N$89: IC4A.IN+, R120.2
- removed net N$90: IC4A.IN-, R68.2, R69.1
- removed net N$91: C140.+, P5.6
- removed net N$93: C156.+, IC4A.OUT, R69.2
- new net N$1: IC3A.IN+, P1.1
- new net N$10: IC2A.IN+, P1.4
- new net N$11: C7.+, P1.5
- new net N$2: IC3A.IN-, IC3A.OUT, IC3B.IN+
- new net N$3: C2.+, IC3B.OUT, R1.2
- new net N$33: IC2A.IN-, IC2A.OUT, IC2B.IN+
- new net N$4: IC3B.IN-, R1.1, R2.2
- new net N$41: C5.+, IC2B.OUT, R8.2
- new net N$47: IC2B.IN-, R8.1, R9.2
- new net N$8: C1.+, P1.6
- net +5VA: now also C3.2, C6.2, IC2P.V+, IC3P.V+; no longer C155.2, C158.2, C195.2, IC10P.V+, IC12P.V+, IC4P.V+, R156.2, R158.2
- net AGND: now also C3.1, C6.1, IC2P.V-, IC3P.V-, R10.1, R3.1; no longer C155.1, C158.1, C192.1, C193.1, C195.1, IC10P.V-, IC12P.V-, IC4P.V-, R121.1, R128.1, R157.1, R159.1
- net OUT-VREF: now also P1.2, P1.3, R2.1, R9.1; no longer IC12A.IN-, IC12A.OUT, P5.2, P5.3, R119.1, R120.1, R126.1, R127.1
- net OUT1-LB: now also C7.-; no longer C160.-
- net OUT1-L^: now also C5.-, R10.2; no longer C157.-, R128.2
- net OUT1-RB: now also C1.-; no longer C140.-
- net OUT1-R^: now also C2.-, R3.2; no longer C141.-, R121.2
