File: circuit/aleph-dev/aleph-primary130808.brd (EAGLE design)
At the start: 174 x 110.5 mm, 379 parts, among them IC10 AD8606, IC12 AD8606, IC2 AD8606, IC3 AD8606, IC4 AD8606, IC5 AD8607R, IC8 AD8607R, IC9 AD8606, J1 STEREOSW2GND, J11 USBA-VERT, J2 NSJ12HF, J20 F-2X03-DIL-100, J21 STEREOSW2GND, J22 STEREOSW2GND, J3 NSJ12HF, J4 NSJ12HF, J5 NSJ12HF, J6 SJ1-3533NG, J8 PJ-102AH/BH, J9 PHA2U, P1 M-1X05-SIP-100-32, P6 F-2X06-DIL-100, P8 M-2X14-DIL-100, SW1 PANASONIC-EVQ, U1 BAS70-04, U10 FDS9431A, U15 AT32UC3A0512, U16 CY62167EV30-Z, U17 AD1939, U2 LMR62014, U23 MT48LC32M16A2tg-75, U24 AD5686R, U26 SN74LVC2G14, U3 BAS70-04, U4 TPS2020, U5 LM2678, U6 ATMEGA32U4-AU, U7 ADP3339, U8 TPA6111A2, U9 ADP3339, X1 16mhz, Y1 ASFL1-27mhz, Y2 12mhz, Y3 ASFL1-12.288mhz

Commit message: circuits and mechanicals
Parts:
- IC5: value AD8607R -> AD8606
Changed lines of the file:
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@@
 <layers>
 <layer number="1" name="Top" color="4" fill="1" visible="yes" active="yes"/>
-<layer number="2" name="power" color="1" fill="3" visible="yes" active="yes"/>
-<layer number="3" name="gnd" color="4" fill="3" visible="yes" active="yes"/>
+<layer number="2" name="power" color="1" fill="3" visible="no" active="yes"/>
+<layer number="3" name="gnd" color="4" fill="3" visible="no" active="yes"/>
 <layer number="4" name="Route4" color="1" fill="4" visible="no" active="no"/>
 <layer number="5" name="Route5" color="4" fill="4" visible="no" active="no"/>
@@
 <layer number="17" name="Pads" color="2" fill="1" visible="yes" active="yes"/>
 <layer number="18" name="Vias" color="2" fill="1" visible="yes" active="yes"/>
-<layer number="19" name="Unrouted" color="6" fill="1" visible="no" active="yes"/>
+<layer number="19" name="Unrouted" color="6" fill="1" visible="yes" active="yes"/>
 <layer number="20" name="Dimension" color="13" fill="1" visible="yes" active="yes"/>
 <layer number="21" name="tPlace" color="7" fill="1" visible="yes" active="yes"/>
 <layer number="22" name="bPlace" color="7" fill="1" visible="no" active="yes"/>
 <layer number="23" name="tOrigins" color="15" fill="1" visible="yes" active="yes"/>
-<layer number="24" name="bOrigins" color="15" fill="1" visible="yes" active="yes"/>
-<layer number="25" name="tNames" color="7" fill="1" visible="yes" active="yes"/>
+<layer number="24" name="bOrigins" color="15" fill="1" visible="no" active="yes"/>
+<layer number="25" name="tNames" color="7" fill="1" visible="no" active="yes"/>
 <layer number="26" name="bNames" color="7" fill="1" visible="no" active="yes"/>
-<layer number="27" name="tValues" color="7" fill="1" visible="no" active="yes"/>
+<layer number="27" name="tValues" color="7" fill="1" visible="yes" active="yes"/>
 <layer number="28" name="bValues" color="7" fill="1" visible="no" active="yes"/>
 <layer number="29" name="tStop" color="7" fill="3" visible="no" active="yes"/>
@@
 <layer number="49" name="Reference" color="7" fill="1" visible="no" active="yes"/>
 <layer number="50" name="dxf" color="7" fill="1" visible="no" active="yes"/>
-<layer number="51" name="tDocu" color="7" fill="1" visible="yes" active="yes"/>
+<layer number="51" name="tDocu" color="7" fill="1" visible="no" active="yes"/>
 <layer number="52" name="bDocu" color="7" fill="1" visible="no" active="yes"/>
 <layer number="53" name="tGND_GNDA" color="7" fill="9" visible="no" active="yes"/>
@@
 <attribute name="VALUE" x="4.1275" y="75.0887" size="0.8128" layer="27" ratio="10"/>
 </element>
-<element name="IC5" library="analog-devices" package="SO8" value="AD8607R" x="11.43" y="70.1675" smashed="yes" rot="R270">
+<element name="IC5" library="analog-devices" package="SO8" value="AD8606" x="11.43" y="70.1675" smashed="yes" rot="R270">
 <attribute name="OC_NEWARK" value="19M8927" x="12.7" y="70.1675" size="1.778" layer="27" rot="R270" display="off"/>
 <attribute name="MPN" value="AD8607ARMZ-R2" x="12.7" y="70.1675" size="1.778" layer="27" rot="R270" display="off"/>
@@
 </signal>
 </signals>
-<errors>
-</errors>
 </board>
 </drawing>
